Commit message: wrong fix, but uploading for now

File: src/Dual_Arm_ROS_Simulation/urdf/dual_arm.xacro (robot description, xacro)
@@ -846,4 +846,42 @@
     </sensor>
   </gazebo>
+  <gazebo reference="L_EE">
+    <mu1>100.0</mu1>
+    <mu2>100.0</mu2>
+    <kp>1000000.0</kp>
+    <kd>100.0</kd>
+    <minDepth>0.003</minDepth>
+    <maxVel>0.0</maxVel>
+    <sensor name="left_contact_sensor" type="contact">
+      <always_on>true</always_on>
+      <update_rate>50.0</update_rate>
+      <contact>
+        <collision>L_EE_collision</collision>
+      </contact>
+      <plugin name="left_bumper" filename="libgazebo_ros_bumper.so">
+        <bumperTopicName>/dual_arm/left_force</bumperTopicName>
+        <frameName>L_EE</frameName>
+      </plugin>
+    </sensor>
+  </gazebo>
+  <gazebo reference="R_EE">
+    <mu1>100.0</mu1>
+    <mu2>100.0</mu2>
+    <kp>1000000.0</kp>
+    <kd>100.0</kd>
+    <minDepth>0.003</minDepth>
+    <maxVel>0.0</maxVel>
+    <sensor name="right_contact_sensor" type="contact">
+      <always_on>true</always_on>
+      <update_rate>50.0</update_rate>
+      <contact>
+        <collision>R_EE_collision</collision>
+      </contact>
+      <plugin name="right_bumper" filename="libgazebo_ros_bumper.so">
+        <bumperTopicName>/dual_arm/right_force</bumperTopicName>
+        <frameName>R_EE</frameName>
+      </plugin>
+    </sensor>
+  </gazebo>
   <gazebo>
     <plugin name="gazebo_ros_control" filename="libgazebo_ros_control.so">

Commit message: Switch grasp control to admittance

File: src/Dual_Arm_ROS_Simulation/urdf/dual_arm.xacro (robot description, xacro)
@@ -407,29 +407,4 @@
       </material>
     </visual>
-    <!-- L자형 턱(lip): 패드는 마찰(μN)에만 의존하므로 접촉 예산 자체는 늘려주지 않는다. 물체
-         아래 모서리를 기하학적으로 받칠 수 있도록 패드 아래쪽에 1cm 턱을 추가한다.
-         로컬축 매핑(위 pick 자세 FK 실측): 로컬 +X가 월드 +Z(수직, dot~0.97)와 거의 나란하고
-         로컬 Y가 스퀴즈 방향이다 - 그래서 "아래"는 로컬 -X, "물체 쪽으로 더 뻗기"는 로컬 -Y다.
-         패드 바닥(로컬 x=-0.02) 바로 아래, 패드 바깥면(로컬 y=-0.0425)보다 1cm 더 뻗어나가게
-         배치해서 물체가 미끄러져 내려오면 이 턱에 걸리도록 한다. -->
-    <collision name="L_EE_grip_lip_collision">
-      <origin
-        xyz="-0.025 -0.0475 -0.005"
-        rpy="0 0 0" />
-      <geometry>
-        <box size="0.01 0.01 0.04" />
-      </geometry>
-    </collision>
-    <visual name="L_EE_grip_lip_visual">
-      <origin
-        xyz="-0.025 -0.0475 -0.005"
-        rpy="0 0 0" />
-      <geometry>
-        <box size="0.01 0.01 0.04" />
-      </geometry>
-      <material name="grip_pad_visual_dark">
-        <color rgba="0.12 0.12 0.12 1" />
-      </material>
-    </visual>
   </link>
   <joint
@@ -744,26 +719,4 @@
       <geometry>
         <box size="0.04 0.01 0.04" />
-      </geometry>
-      <material name="grip_pad_visual_dark">
-        <color rgba="0.12 0.12 0.12 1" />
-      </material>
-    </visual>
-    <!-- L자형 턱(lip) - L_EE 쪽 설명/축 매핑 참고 (R도 로컬 +X가 월드 +Z와 dot~0.97로 거의
-         나란함). 패드 바닥(로컬 x=-0.02) 아래, 패드 바깥면(로컬 y=0.0425)보다 1cm 더 뻗어나가게
-         배치. -->
-    <collision name="R_EE_grip_lip_collision">
-      <origin
-        xyz="-0.025 0.0475 -0.005"
-        rpy="0 0 0" />
-      <geometry>
-        <box size="0.01 0.01 0.04" />
-      </geometry>
-    </collision>
-    <visual name="R_EE_grip_lip_visual">
-      <origin
-        xyz="-0.025 0.0475 -0.005"
-        rpy="0 0 0" />
-      <geometry>
-        <box size="0.01 0.01 0.04" />
       </geometry>
       <material name="grip_pad_visual_dark">

Commit message: Tune dual-arm grasp approach and face-contact gating

File: src/Dual_Arm_ROS_Simulation/urdf/dual_arm.xacro (robot description, xacro)
@@ -393,5 +393,5 @@
         rpy="0 0 0" />
       <geometry>
-        <box size="0.04 0.01 0.04" />
+        <box size="0.055 0.014 0.055" />
       </geometry>
     </collision>
@@ -401,5 +401,5 @@
         rpy="0 0 0" />
       <geometry>
-        <box size="0.04 0.01 0.04" />
+        <box size="0.055 0.014 0.055" />
       </geometry>
       <material name="grip_pad_visual_dark">
@@ -710,5 +710,5 @@
         rpy="0 0 0" />
       <geometry>
-        <box size="0.04 0.01 0.04" />
+        <box size="0.055 0.014 0.055" />
       </geometry>
     </collision>
@@ -718,5 +718,5 @@
         rpy="0 0 0" />
       <geometry>
-        <box size="0.04 0.01 0.04" />
+        <box size="0.055 0.014 0.055" />
       </geometry>
       <material name="grip_pad_visual_dark">
@@ -912,7 +912,19 @@
     <provideFeedback>true</provideFeedback>
   </gazebo>
+  <gazebo reference="L_EE">
+    <mu1>3.0</mu1>
+    <mu2>3.0</mu2>
+    <kp>1000000.0</kp>
+    <kd>10.0</kd>
+  </gazebo>
   <gazebo reference="R_EE_joint">
     <disableFixedJointLumping>true</disableFixedJointLumping>
     <provideFeedback>true</provideFeedback>
+  </gazebo>
+  <gazebo reference="R_EE">
+    <mu1>3.0</mu1>
+    <mu2>3.0</mu2>
+    <kp>1000000.0</kp>
+    <kd>10.0</kd>
   </gazebo>
   <!-- gazebo_ros_ft_sensor: L_EE_joint/R_EE_joint에 걸리는 반력을 각각
