Commit message: Added 2DOF Head

File: src/Dual_Arm_ROS_Simulation/urdf/dual_arm.urdf (robot description, URDF)
Before this commit: robot dual_arm, 24 links, 23 joints
Links:
- added link Neck_link, mass 0.05
Joints:
- removed joint Head_joint
- added joint Head_pitch_joint: type revolute, parent Neck_link, child Head, origin xyz=0 0 0 rpy=0 0 0, axis 0 1 0, limit lower=-1.0 upper=1.0 effort=30 velocity=5
- added joint Head_yaw_joint: type revolute, parent Torso, child Neck_link, origin xyz=-0.0027205 0 0.45287 rpy=0 0 0, axis 0 0 1, limit lower=-1.57 upper=1.57 effort=30 velocity=5

File: src/Dual_Arm_ROS_Simulation/urdf/dual_arm.xacro (robot description, xacro)
@@ -1,5 +1,5 @@
 <?xml version="1.0" ?>
 <robot name="dual_arm" xmlns:xacro="http://www.ros.org/wiki/xacro">
-<link name="world"/>
+  <link name="world"/>
   <joint name="fixed" type="fixed">
     <parent link="world"/>
@@ -7,695 +7,380 @@
     <origin rpy="0 0 0" xyz="0 0 0.86"/>
   </joint>
-  <link
-    name="Pelvis">
-    <inertial>
-      <origin
-        xyz="-4E-06 1E-05 0.030876"
-        rpy="0 0 0" />
-      <mass
-        value="5.123963" />
-      <inertia
-        ixx="0.051784"
-        ixy="0"
-        ixz="1E-06"
-        iyy="0.01018"
-        iyz="-1E-06"
-        izz="0.055756" />
-    </inertial>
-    <visual>
-      <origin
-        xyz="0 0 0"
-        rpy="0 0 0" />
-      <geometry>
-        <mesh
-          filename="package://dual_arm/meshes/Pelvis.STL" />
-      </geometry>
-      <material
-        name="">
-        <color
-          rgba="0.792156862745098 0.819607843137255 0.933333333333333 1" />
-      </material>
-    </visual>
-    <collision>
-      <origin
-        xyz="0 0 0"
-        rpy="0 0 0" />
-      <geometry>
-        <mesh
-          filename="package://dual_arm/meshes/Pelvis.STL" />
-      </geometry>
-    </collision>
-  </link>
-  <link
-    name="Torso">
-    <inertial>
-      <origin
-        xyz="-0.004339 0 0.216108"
-        rpy="0 0 0" />
-      <mass
-        value="16.636925" />
-      <inertia
-        ixx="0.296782"
-        ixy="-2.9E-05"
-        ixz="-0.0052"
-        iyy="0.232939"
-        iyz="0"
-        izz="0.114483" />
-    </inertial>
-    <visual>
-      <origin
-        xyz="0 0 0"
-        rpy="0 0 0" />
-      <geometry>
-        <mesh
-          filename="package://dual_arm/meshes/Torso.STL" />
-      </geometry>
-      <material
-        name="">
-        <color
-          rgba="0.792156862745098 0.819607843137255 0.933333333333333 1" />
-      </material>
-    </visual>
-    <collision>
-      <origin
-        xyz="0 0 0"
-        rpy="0 0 0" />
-      <geometry>
-        <mesh
-          filename="package://dual_arm/meshes/Torso.STL" />
-      </geometry>
-    </collision>
-  </link>
-  <joint
-    name="Waist_joint"
-    type="revolute">
-    <origin
-      xyz="0 0 0.0825"
-      rpy="0 0 0" />
-    <parent
-      link="Pelvis" />
-    <child
-      link="Torso" />
-    <axis
-      xyz="0 0 1" />
-    <dynamics damping="1"/>
-    <limit
-      lower="-0.87"
-      upper="0.87"
-      effort="100"
-      velocity="13" />
-  </joint>
-  <link
-    name="L_shoulder_pitch">
-    <inertial>
-      <origin
-        xyz="0.010378 0.049076 0"
-        rpy="0 0 0" />
-      <mass
-        value="0.47258" />
-      <inertia
-        ixx="0.000904"
-        ixy="6.4E-05"
-        ixz="0"
-        iyy="0.000955"
-        iyz="0"
-        izz="0.001372" />
-    </inertial>
-    <visual>
-      <origin
-        xyz="0 0 0"
-        rpy="0 0 0" />
-      <geometry>
-        <mesh
-          filename="package://dual_arm/meshes/L_shoulder_pitch.STL" />
-      </geometry>
-      <material
-        name="">
-        <color
-          rgba="0.79216 0.81961 0.93333 1" />
-      </material>
-    </visual>
-    <collision>
-      <origin
-        xyz="0 0 0"
-        rpy="0 0 0" />
-      <geometry>
-        <mesh
-          filename="package://dual_arm/meshes/L_shoulder_pitch.STL" />
-      </geometry>
-    </collision>
-  </link>
-  <joint
-    name="L_shoulder_pitch_joint"
-    type="revolute">
-    <origin
-      xyz="-0.0082603 0.16 0.36224"
-      rpy="0.34907 0 0" />
-    <parent
-      link="Torso" />
-    <child
-      link="L_shoulder_pitch" />
-    <axis
-      xyz="0 1 0" />
-    <dynamics damping="1"/>
-    <limit
-      lower="-3.14"
-      upper="1.05"
-      effort="55"
-      velocity="16" />
-  </joint>
-  <link
-    name="L_shoulder_roll">
-    <inertial>
-      <origin
-        xyz="0.001469 -7E-05 -0.079989"
-        rpy="0 0 0" />
-      <mass
-        value="2.002576" />
-      <inertia
-        ixx="0.020339"
-        ixy="-4E-06"
-        ixz="0.000225"
-        iyy="0.020072"
-        iyz="4.8E-05"
-        izz="0.002315" />
-    </inertial>
-    <visual>
-      <origin
-        xyz="0 0 0"
-        rpy="0 0 0" />
-      <geometry>
-        <mesh
-          filename="package://dual_arm/meshes/L_shoulder_roll.STL" />
-      </geometry>
-      <material
-        name="">
-        <color
-          rgba="0.792156862745098 0.819607843137255 0.933333333333333 1" />
-      </material>
-    </visual>
-    <collision>
-      <origin
-        xyz="0 0 0"
-        rpy="0 0 0" />
-      <geometry>
-        <mesh
-          filename="package://dual_arm/meshes/L_shoulder_roll.STL" />
-      </geometry>
-    </collision>
-  </link>
-  <joint
-    name="L_shoulder_roll_joint"
-    type="revolute">
-    <origin
-      xyz="0.0082603 0.082 0"
-      rpy="-0.261799387799 0 0" />
-    <parent
-      link="L_shoulder_pitch" />
-    <child
-      link="L_shoulder_roll" />
-    <axis
-      xyz="1 0 0" />
-    <dynamics damping="1"/>
-    <limit
-      lower="-0.349"
-      upper="2.62"
-      effort="55"
-      velocity="16" />
-  </joint>
-  <link
-    name="L_shoulder_yaw">
-    <inertial>
-      <origin
-        xyz="4.8E-05 0.00162 -0.045384"
-        rpy="0 0 0" />
-      <mass
-        value="0.608514" />
-      <inertia
-        ixx="0.000608"
-        ixy="0"
-        ixz="0"
-        iyy="0.00049"
-        iyz="-2E-06"
-        izz="0.000483" />
-    </inertial>
-    <visual>
-      <origin
-        xyz="0 0 0"
-        rpy="0 0 0" />
-      <geometry>
-        <mesh
-          filename="package://dual_arm/meshes/L_shoulder_yaw.STL" />
-      </geometry>
-      <material
-        name="">
-        <color
-          rgba="0.792156862745098 0.819607843137255 0.933333333333333 1" />
-      </material>
-    </visual>
-    <collision>
-      <origin
-        xyz="0 0 0"
-        rpy="0 0 0" />
-      <geometry>
-        <mesh
-          filename="package://dual_arm/meshes/L_shoulder_yaw.STL" />
-      </geometry>
-    </collision>
-  </link>
-  <joint
-    name="L_shoulder_yaw_joint"
-    type="revolute">
-    <origin
-      xyz="0 0 -0.2505"
-      rpy="0 0 0" />
-    <parent
-      link="L_shoulder_roll" />
-    <child
-      link="L_shoulder_yaw" />
-    <axis
-      xyz="0 0 1" />
-    <dynamics damping="1"/>
-    <limit
-      lower="-1.57"
-      upper="1.57"
-      effort="30"
-      velocity="8.5" />
-  </joint>
-  <link
-    name="L_elbow">
-    <inertial>
-      <origin
-        xyz="0 -5.2E-05 -0.075944"
-        rpy="0 0 0" />
-      <mass
-        value="0.297153" />
-      <inertia
-        ixx="0.001705"
-        ixy="0"
-        ixz="0"
-        iyy="0.001534"
-        iyz="-1E-06"
-        izz="0.000304" />
-    </inertial>
-    <visual>
-      <origin
-        xyz="0 0 0"
-        rpy="0 0 0" />
-      <geometry>
-        <mesh
-          filename="package://dual_arm/meshes/L_elbow.STL" />
-      </geometry>
-      <material
-        name="">
-        <color
-          rgba="0.792156862745098 0.819607843137255 0.933333333333333 1" />
-      </material>
-    </visual>
-    <collision>
-      <origin
-        xyz="0 0 0"
-        rpy="0 0 0" />
-      <geometry>
-        <mesh
-          filename="package://dual_arm/meshes/L_elbow.STL" />
-      </geometry>
-    </collision>
-  </link>
-  <joint
-    name="L_elbow_joint"
-    type="revolute">
-    <origin
-      xyz="0 0 -0.0545"
-      rpy="0 0 0" />
-    <parent
-      link="L_shoulder_yaw" />
-    <child
-      link="L_elbow" />
-    <axis
-      xyz="0 1 0" />
-    <dynamics damping="1"/>
-    <limit
-      lower="-1.9"
-      upper="1.05"
-      effort="30"
-      velocity="8.5" />
-  </joint>
-  <link
-    name="L_EE">
-    <inertial>
-      <origin
-        xyz="0 0 -0.003514"
-        rpy="0 0 0" />
-      <mass
-        value="0.15" />
-      <inertia
-        ixx="5.5E-05"
-        ixy="0"
-        ixz="0"
-        iyy="5.5E-05"
-        iyz="0"
-        izz="6.4E-05" />
-    </inertial>
-    <visual>
-      <origin
-        xyz="0 0 0"
-        rpy="0 0 0" />
-      <geometry>
-        <mesh
-          filename="package://dual_arm/meshes/L_EE.STL" />
-      </geometry>
-      <material
-        name="">
-        <color
-          rgba="0.298039215686275 0.298039215686275 0.298039215686275 1" />
-      </material>
-    </visual>
-    <collision>
-      <origin
-        xyz="0 0 0"
-        rpy="0 0 0" />
-      <geometry>
-        <mesh
-          filename="package://dual_arm/meshes/L_EE.STL" />
-      </geometry>
-    </collision>
-  </link>
-  <joint
-    name="L_EE_joint"
-    type="fixed">
-    <origin
-      xyz="0 0 -0.3"
-      rpy="0 0 0" />
-    <parent
-      link="L_elbow" />
-    <child
-      link="L_EE" />
-    <axis
-      xyz="0 0 0" />
-    <dynamics damping="1"/>
-    <limit
-      lower="-1.57"
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