Commit message: Refine dual-arm pick place workspace and split IK

File: src/Dual_Arm_ROS_Simulation/urdf/dual_arm.urdf (robot description, URDF)
Before this commit: robot dual_arm, 25 links, 24 joints
Links:
- removed link Neck_link
- added link Head_camera_link, mass 0.05; visual sphere radius=0.02
- added link Head_camera_link_optical
- added link Head_yaw_link, mass 0.01
Joints:
- added joint Head_camera_joint: type fixed, parent Head, child Head_camera_link, origin xyz=0.05 0 0.145 rpy=0 0 0
- added joint Head_camera_optical_joint: type fixed, parent Head_camera_link, child Head_camera_link_optical, origin xyz=0 0 0 rpy=-1.5707963 0 -1.5707963
- joint Head_pitch_joint: limit lower=-1.0 upper=1.0 effort=30 velocity=5 -> lower=-0.5236 upper=0.5236 effort=10 velocity=8.5; parent Neck_link -> Head_yaw_link
- joint Head_yaw_joint: child Neck_link -> Head_yaw_link; limit lower=-1.57 upper=1.57 effort=30 velocity=5 -> lower=-1.2217 upper=1.2217 effort=10 velocity=8.5
- joint L_shoulder_pitch_joint: origin xyz=-0.0082603 0.16 0.36224 rpy=0.34907 0 0 -> xyz=-0.0082603 0.16 0.36224 rpy=0.34907 -1.57079632679 0
- joint R_shoulder_pitch_joint: origin xyz=-0.0082603 -0.16 0.36224 rpy=-0.34907 0 0 -> xyz=-0.0082603 -0.16 0.36224 rpy=-0.34907 -1.57079632679 0

File: src/Dual_Arm_ROS_Simulation/urdf/dual_arm.xacro (robot description, xacro)
@@ -1,5 +1,5 @@
 <?xml version="1.0" ?>
 <robot name="dual_arm" xmlns:xacro="http://www.ros.org/wiki/xacro">
-  <link name="world"/>
+<link name="world"/>
   <joint name="fixed" type="fixed">
     <parent link="world"/>
@@ -7,380 +7,746 @@
     <origin rpy="0 0 0" xyz="0 0 0.86"/>
   </joint>
-  <link name="Pelvis">
-    <inertial>
-      <origin xyz="-4E-06 1E-05 0.030876" rpy="0 0 0" />
-      <mass value="5.123963" />
-      <inertia ixx="0.051784" ixy="0" ixz="1E-06" iyy="0.01018" iyz="-1E-06" izz="0.055756" />
-    </inertial>
-    <visual>
-      <origin xyz="0 0 0" rpy="0 0 0" />
-      <geometry>
-        <mesh filename="package://dual_arm/meshes/Pelvis.STL" />
-     </geometry>
-      <material name="">
-        <color rgba="0.792156862745098 0.819607843137255 0.933333333333333 1" />
-      </material>
-    </visual>
-    <collision>
-      <origin xyz="0 0 0" rpy="0 0 0" />
-      <geometry>
-        <mesh filename="package://dual_arm/meshes/Pelvis.STL" />
-      </geometry>
-    </collision>
-  </link>
-  <link name="Torso">
-    <inertial>
-      <origin xyz="-0.004339 0 0.216108" rpy="0 0 0" />
-      <mass value="16.636925" />
-      <inertia ixx="0.296782" ixy="-2.9E-05" ixz="-0.0052" iyy="0.232939" iyz="0" izz="0.114483" />
-    </inertial>
-    <visual>
-      <origin xyz="0 0 0" rpy="0 0 0" />
-      <geometry>
-        <mesh filename="package://dual_arm/meshes/Torso.STL" />
-      </geometry>
-      <material name="">
-        <color rgba="0.792156862745098 0.819607843137255 0.933333333333333 1" />
-      </material>
-    </visual>
-    <collision>
-      <origin xyz="0 0 0" rpy="0 0 0" />
-      <geometry>
-        <mesh filename="package://dual_arm/meshes/Torso.STL" />
-      </geometry>
-    </collision>
-  </link>
-  <joint name="Waist_joint" type="revolute">
-    <origin xyz="0 0 0.0825" rpy="0 0 0" />
-    <parent link="Pelvis" />
-    <child link="Torso" />
-    <axis xyz="0 0 1" />
-    <dynamics damping="1"/>
-    <limit lower="-0.87" upper="0.87" effort="100" velocity="13" />
-  </joint>
-  <link name="L_shoulder_pitch">
-    <inertial>
-      <origin xyz="0.010378 0.049076 0" rpy="0 0 0" />
-      <mass value="0.47258" />
-      <inertia ixx="0.000904" ixy="6.4E-05" ixz="0" iyy="0.000955" iyz="0" izz="0.001372" />
-    </inertial>
-    <visual>
-      <origin xyz="0 0 0" rpy="0 0 0" />
-      <geometry>
-        <mesh filename="package://dual_arm/meshes/L_shoulder_pitch.STL" />
-      </geometry>
-      <material name="">
-         <color rgba="0.79216 0.81961 0.93333 1" />
-      </material>
-    </visual>
-    <collision>
-      <origin xyz="0 0 0" rpy="0 0 0" />
-      <geometry>
-        <mesh filename="package://dual_arm/meshes/L_shoulder_pitch.STL" />
-      </geometry>
-    </collision>
-  </link>
-  <joint name="L_shoulder_pitch_joint" type="revolute">
-    <origin xyz="-0.0082603 0.16 0.36224" rpy="0.34907 0 0" />
-    <parent link="Torso" />
-    <child link="L_shoulder_pitch" />
-    <axis xyz="0 1 0" />
-    <dynamics damping="1"/>
-    <limit lower="-3.14" upper="1.05" effort="55" velocity="16" />
-  </joint>
-  <link name="L_shoulder_roll">
-    <inertial>
-      <origin xyz="0.001469 -7E-05 -0.079989" rpy="0 0 0" />
-      <mass value="2.002576" />
-      <inertia ixx="0.020339" ixy="-4E-06" ixz="0.000225" iyy="0.020072" iyz="4.8E-05" izz="0.002315" />
-    </inertial>
-    <visual>
-      <origin xyz="0 0 0" rpy="0 0 0" />
-      <geometry>
-        <mesh filename="package://dual_arm/meshes/L_shoulder_roll.STL" />
-      </geometry>
-      <material name="">
-        <color rgba="0.792156862745098 0.819607843137255 0.933333333333333 1" />
-      </material>
-    </visual>
-    <collision>
-      <origin xyz="0 0 0" rpy="0 0 0" />
-      <geometry>
-        <mesh filename="package://dual_arm/meshes/L_shoulder_roll.STL" />
-      </geometry>
-    </collision>
-  </link>
-  <joint name="L_shoulder_roll_joint" type="revolute">
-    <origin xyz="0.0082603 0.082 0" rpy="-0.261799387799 0 0" />
-    <parent link="L_shoulder_pitch" />
-    <child link="L_shoulder_roll" />
-    <axis xyz="1 0 0" />
-    <dynamics damping="1"/>
-    <limit lower="-0.349" upper="2.62" effort="55" velocity="16" />
-  </joint>
-  <link name="L_shoulder_yaw">
-    <inertial>
-      <origin xyz="4.8E-05 0.00162 -0.045384" rpy="0 0 0" />
-      <mass value="0.608514" />
-      <inertia ixx="0.000608" ixy="0" ixz="0" iyy="0.00049" iyz="-2E-06" izz="0.000483" />
-    </inertial>
-    <visual>
-      <origin xyz="0 0 0" rpy="0 0 0" />
-      <geometry>
-        <mesh filename="package://dual_arm/meshes/L_shoulder_yaw.STL" />
-      </geometry>
-      <material name="">
-        <color rgba="0.792156862745098 0.819607843137255 0.933333333333333 1" />
-      </material>
-    </visual>
-    <collision>
-      <origin xyz="0 0 0" rpy="0 0 0" />
-      <geometry>
-        <mesh filename="package://dual_arm/meshes/L_shoulder_yaw.STL" />
-      </geometry>
-    </collision>
-  </link>
-  <joint name="L_shoulder_yaw_joint" type="revolute">
-    <origin xyz="0 0 -0.2505" rpy="0 0 0" />
-    <parent link="L_shoulder_roll" />
-    <child link="L_shoulder_yaw" />
-    <axis xyz="0 0 1" />
-    <dynamics damping="1"/>
-    <limit lower="-1.57" upper="1.57" effort="30" velocity="8.5" />
-  </joint>
-  <link name="L_elbow">
-    <inertial>
-      <origin xyz="0 -5.2E-05 -0.075944" rpy="0 0 0" />
-      <mass value="0.297153" />
-      <inertia ixx="0.001705" ixy="0" ixz="0" iyy="0.001534" iyz="-1E-06" izz="0.000304" />
-    </inertial>
-    <visual>
-      <origin xyz="0 0 0" rpy="0 0 0" />
-      <geometry>
-        <mesh filename="package://dual_arm/meshes/L_elbow.STL" />
-      </geometry>
-      <material name="">
-        <color rgba="0.792156862745098 0.819607843137255 0.933333333333333 1" />
-      </material>
-    </visual>
-    <collision>
-      <origin xyz="0 0 0" rpy="0 0 0" />
-      <geometry>
-        <mesh filename="package://dual_arm/meshes/L_elbow.STL" />
-      </geometry>
-    </collision>
-  </link>
-  <joint name="L_elbow_joint" type="revolute">
-    <origin xyz="0 0 -0.0545" rpy="0 0 0" />
-    <parent link="L_shoulder_yaw" />
-    <child link="L_elbow" />
-    <axis xyz="0 1 0" />
-    <dynamics damping="1"/>
-    <limit lower="-1.9" upper="1.05" effort="30" velocity="8.5" />
-  </joint>
-  <link name="L_EE">
-    <inertial>
-      <origin xyz="0 0 -0.003514" rpy="0 0 0" />
-      <mass value="0.15" />
-      <inertia ixx="5.5E-05" ixy="0" ixz="0" iyy="5.5E-05" iyz="0" izz="6.4E-05" />
-    </inertial>
-    <visual>
-      <origin xyz="0 0 0" rpy="0 0 0" />
-      <geometry>
-        <mesh filename="package://dual_arm/meshes/L_EE.STL" />
-      </geometry>
-      <material name="">
-        <color rgba="0.298039215686275 0.298039215686275 0.298039215686275 1" />
-      </material>
-    </visual>
-    <collision>
-      <origin xyz="0 0 0" rpy="0 0 0" />
-      <geometry>
-        <mesh filename="package://dual_arm/meshes/L_EE.STL" />
-      </geometry>
-    </collision>
-  </link>
-  <joint name="L_EE_joint" type="fixed">
-    <origin xyz="0 0 -0.3" rpy="0 0 0" />
-    <parent link="L_elbow" />
-    <child link="L_EE" />
-    <axis xyz="0 0 0" />
-    <dynamics damping="1"/>
-    <limit lower="-1.57" upper="1.57" effort="30" velocity="8.5" />
-  </joint>
-  <link name="R_shoulder_pitch">
-    <inertial>
-      <origin xyz="0.010378 -0.049076 0" rpy="0 0 0" />
-      <mass value="0.472578" />
-      <inertia ixx="0.000904" ixy="-6.4E-05" ixz="0" iyy="0.000955" iyz="0" izz="0.001372" />
-    </inertial>
-    <visual>
-      <origin xyz="0 0 0" rpy="0 0 0" />
-      <geometry>
-        <mesh filename="package://dual_arm/meshes/R_shoulder_pitch.STL" />
-      </geometry>
-      <material name="">
-        <color rgba="0.792156862745098 0.819607843137255 0.933333333333333 1" />
-      </material>
-    </visual>
-    <collision>
-      <origin xyz="0 0 0" rpy="0 0 0" />
-      <geometry>
-        <mesh filename="package://dual_arm/meshes/R_shoulder_pitch.STL" />
-      </geometry>
-    </collision>
-  </link>
-  <joint name="R_shoulder_pitch_joint" type="revolute">
-    <origin xyz="-0.0082603 -0.16 0.36224" rpy="-0.34907 0 0" />
-    <parent link="Torso" />
-    <child link="R_shoulder_pitch" />
-    <axis xyz="0 1 0" />
-    <dynamics damping="1"/>
-    <limit lower="-3.14" upper="1.05" effort="55" velocity="16" />
-  </joint>
-  <link name="R_shoulder_roll">
-    <inertial>
-      <origin xyz="0.001469 -7E-05 -0.079989" rpy="0 0 0" />
-      <mass value="2.002576" />
-      <inertia ixx="0.020339" ixy="-4E-06" ixz="0.000225" iyy="0.020072" iyz="4.8E-05" izz="0.002315" />
-    </inertial>
-    <visual>
-      <origin xyz="0 0 0" rpy="0 0 0" />
-      <geometry>
-        <mesh filename="package://dual_arm/meshes/R_shoulder_roll.STL" />
-      </geometry>
-      <material name="">
-        <color rgba="0.792156862745098 0.819607843137255 0.933333333333333 1" />
-      </material>
-    </visual>
-    <collision>
-      <origin xyz="0 0 0" rpy="0 0 0" />
-      <geometry>
-        <mesh filename="package://dual_arm/meshes/R_shoulder_roll.STL" />
-      </geometry>
-    </collision>
-  </link>
-  <joint name="R_shoulder_roll_joint" type="revolute">
-    <origin xyz="0.0082603 -0.082 0" rpy="0.261799387799 0 0" />
-    <parent link="R_shoulder_pitch" />
-    <child link="R_shoulder_roll" />
-    <axis xyz="1 0 0" />
-    <dynamics damping="1"/>
-    <limit lower="-2.62" upper="0.349" effort="55" velocity="16" />
-  </joint>
-  <link name="R_shoulder_yaw">
-    <inertial>
-      <origin xyz="-4.8E-05 -0.00162 -0.045384" rpy="0 0 0" />
-      <mass value="0.608514" />
-      <inertia ixx="0.000608" ixy="0" ixz="0" iyy="0.00049" iyz="2E-06" izz="0.000483" />
-    </inertial>
-    <visual>
-      <origin xyz="0 0 0" rpy="0 0 0" />
-      <geometry>
-        <mesh filename="package://dual_arm/meshes/R_shoulder_yaw.STL" />
-      </geometry>
-      <material name="">
-        <color rgba="0.792156862745098 0.819607843137255 0.933333333333333 1" />
-      </material>
-    </visual>
-    <collision>
-      <origin xyz="0 0 0" rpy="0 0 0" />
-      <geometry>
-        <mesh filename="package://dual_arm/meshes/R_shoulder_yaw.STL" />
-      </geometry>
-    </collision>
-  </link>
-  <joint name="R_shoulder_yaw_joint" type="revolute">
-    <origin xyz="0 0 -0.2505" rpy="0 0 0" />
-    <parent link="R_shoulder_roll" />
-    <child link="R_shoulder_yaw" />
-    <axis xyz="0 0 1" />
-    <dynamics damping="1"/>
-    <limit lower="-1.57" upper="1.57" effort="30" velocity="8.5" />
-  </joint>
-  <link name="R_elbow">
-    <inertial>
-      <origin xyz="0 5.2E-05 -0.075944" rpy="0 0 0" />
-      <mass value="0.297153" />
-      <inertia ixx="0.001705" ixy="0" ixz="0" iyy="0.001534" iyz="1E-06" izz="0.000304" />
-    </inertial>
-    <visual>
-      <origin xyz="0 0 0" rpy="0 0 0" />
-      <geometry>
-        <mesh filename="package://dual_arm/meshes/R_elbow.STL" />
-      </geometry>
-      <material name="">
-        <color rgba="0.792156862745098 0.819607843137255 0.933333333333333 1" />
-      </material>
-    </visual>
-    <collision>
-      <origin xyz="0 0 0" rpy="0 0 0" />
-      <geometry>
-        <mesh filename="package://dual_arm/meshes/R_elbow.STL" />
-      </geometry>
-    </collision>
-  </link>
-  <joint name="R_elbow_joint" type="revolute">
-    <origin xyz="0 0 -0.0545" rpy="0 0 0" />
-    <parent link="R_shoulder_yaw" />
-    <child link="R_elbow" />
-    <axis xyz="0 1 0" />
-    <dynamics damping="1"/>
-    <limit lower="-1.9" upper="1.05" effort="30" velocity="8.5" />
-  </joint>
-  <link name="R_EE">
-    <inertial>
-      <origin xyz="0 0 -0.003514" rpy="0 0 0" />
-      <mass value="0.15" />
-      <inertia ixx="5.5E-05" ixy="0" ixz="0" iyy="5.5E-05" iyz="0" izz="6.4E-05" />
-    </inertial>
-    <visual>
-      <origin xyz="0 0 0" rpy="0 0 0" />
-      <geometry>
-        <mesh filename="package://dual_arm/meshes/R_EE.STL" />
-      </geometry>
-      <material name="">
-        <color rgba="0.298039215686275 0.298039215686275 0.298039215686275 1" />
-      </material>
-    </visual>
-    <collision>
-      <origin xyz="0 0 0" rpy="0 0 0" />
-      <geometry>
-        <mesh filename="package://dual_arm/meshes/R_EE.STL" />
-      </geometry>
-    </collision>
-  </link>
-  <joint name="R_EE_joint" type="fixed">
-    <origin xyz="0 0 -0.3" rpy="0 0 0" />
-    <parent link="R_elbow" />
-    <child link="R_EE" />
-    <axis xyz="0 0 0" />
-    <dynamics damping="1"/>
-    <limit lower="-1.57" upper="1.57" effort="30" velocity="8.5" />
-  </joint>
-  <link name="Neck_link">
-    <inertial>
-      <origin xyz="0 0 0" rpy="0 0 0"/>
-      <mass value="0.05"/>
-      <inertia ixx="1E-5" ixy="0" ixz="0" iyy="1E-5" iyz="0" izz="1E-5"/>
-    </inertial>
-  </link>
-  <joint name="Head_yaw_joint" type="revolute">
-    <origin xyz="-0.0027205 0 0.45287" rpy="0 0 0" />
-    <parent link="Torso" />
-    <child link="Neck_link" />
-    <axis xyz="0 0 1" />
-    <dynamics damping="1"/>
-    <limit lower="-1.57" upper="1.57" effort="30" velocity="5" />
-  </joint>
-  <joint name="Head_pitch_joint" type="revolute">
-    <origin xyz="0 0 0" rpy="0 0 0" />
-    <parent link="Neck_link" />
-    <child link="Head" />
-    <axis xyz="0 1 0" />
-    <dynamics damping="1"/>
-    <limit lower="-1.0" upper="1.0" effort="30" velocity="5" />
-  </joint>
-  <link name="Head">
+  <link
+    name="Pelvis">
+    <inertial>
+      <origin
+        xyz="-4E-06 1E-05 0.030876"
+        rpy="0 0 0" />
+      <mass
+        value="5.123963" />
+      <inertia
+        ixx="0.051784"
+        ixy="0"
+        ixz="1E-06"
+        iyy="0.01018"
+        iyz="-1E-06"
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
Commit message: Stabilize vision pick-place head scan

File: src/Dual_Arm_ROS_Simulation/urdf/dual_arm.urdf (robot description, URDF)
Before this commit: robot dual_arm, 27 links, 26 joints
Links:
- link L_EE: geometry collision mesh filename=package://dual_arm/meshes/L_EE.STL; visual box size=0.01 0.01 0.04
- link R_EE: geometry collision mesh filename=package://dual_arm/meshes/R_EE.STL; visual box size=0.01 0.01 0.04
Joints:
- joint Head_pitch_joint: limit lower=-0.5236 upper=0.5236 effort=10 velocity=8.5 -> lower=-0.5236 upper=1.0472 effort=10 velocity=8.5

File: src/Dual_Arm_ROS_Simulation/urdf/dual_arm.xacro (robot description, xacro)
@@ -396,4 +396,15 @@
       </geometry>
     </collision>
+    <visual name="L_EE_grip_pad_visual">
+      <origin
+        xyz="0 -0.0375 -0.005"
+        rpy="0 0 0" />
+      <geometry>
+        <box size="0.04 0.01 0.04" />
+      </geometry>
+      <material name="grip_pad_visual_dark">
+        <color rgba="0.12 0.12 0.12 1" />
+      </material>
+    </visual>
     <!-- L자형 턱(lip): 패드는 마찰(μN)에만 의존하므로 접촉 예산 자체는 늘려주지 않는다. 물체
          아래 모서리를 기하학적으로 받칠 수 있도록 패드 아래쪽에 1cm 턱을 추가한다.
@@ -410,4 +421,15 @@
       </geometry>
     </collision>
+    <visual name="L_EE_grip_lip_visual">
+      <origin
+        xyz="-0.025 -0.0475 -0.005"
+        rpy="0 0 0" />
+      <geometry>
+        <box size="0.01 0.01 0.04" />
+      </geometry>
+      <material name="grip_pad_visual_dark">
+        <color rgba="0.12 0.12 0.12 1" />
+      </material>
+    </visual>
   </link>
   <joint
@@ -716,4 +738,15 @@
       </geometry>
     </collision>
+    <visual name="R_EE_grip_pad_visual">
+      <origin
+        xyz="0 0.0375 -0.005"
+        rpy="0 0 0" />
+      <geometry>
+        <box size="0.04 0.01 0.04" />
+      </geometry>
+      <material name="grip_pad_visual_dark">
+        <color rgba="0.12 0.12 0.12 1" />
+      </material>
+    </visual>
     <!-- L자형 턱(lip) - L_EE 쪽 설명/축 매핑 참고 (R도 로컬 +X가 월드 +Z와 dot~0.97로 거의
          나란함). 패드 바닥(로컬 x=-0.02) 아래, 패드 바깥면(로컬 y=0.0425)보다 1cm 더 뻗어나가게
@@ -727,4 +760,15 @@
       </geometry>
     </collision>
+    <visual name="R_EE_grip_lip_visual">
+      <origin
+        xyz="-0.025 0.0475 -0.005"
+        rpy="0 0 0" />
+      <geometry>
+        <box size="0.01 0.01 0.04" />
+      </geometry>
+      <material name="grip_pad_visual_dark">
+        <color rgba="0.12 0.12 0.12 1" />
+      </material>
+    </visual>
   </link>
   <joint
@@ -820,5 +864,5 @@
     <limit
       lower="-0.5236"
-      upper="0.5236"
+      upper="1.0472"
       effort="10"
       velocity="8.5" />
