Commit message: Implement wrist-aware dual-arm grasp control

File: src/Dual_Arm_ROS_Simulation/urdf/dual_arm.urdf (robot description, URDF)
Before this commit: robot dual_arm, 27 links, 26 joints
Links:
- added link L_grip_frame
- added link L_wrist_ik_frame, mass 0.001
- added link L_wrist_yaw, mass 0.5; visual cylinder length=0.03 radius=0.017
- added link R_grip_frame
- added link R_wrist_ik_frame, mass 0.001
- added link R_wrist_yaw, mass 0.5; visual cylinder length=0.03 radius=0.017
- link Head_camera_link: geometry 
- link L_EE: geometry collision box size=0.090 0.025 0.090; visual box size=0.090 0.025 0.090
- link R_EE: geometry collision box size=0.090 0.025 0.090; visual box size=0.090 0.025 0.090
Joints:
- added joint L_grip_joint: type fixed, parent L_EE, child L_grip_frame, origin xyz=0 -0.0375 -0.005 rpy=0 0 0
- added joint L_wrist_ik_joint: type fixed, parent L_wrist_yaw, child L_wrist_ik_frame, origin xyz=0 0 -0.10 rpy=0 0 0
- added joint L_wrist_yaw_joint: type revolute, parent L_elbow, child L_wrist_yaw, origin xyz=0 0 -0.15 rpy=0 0 0, axis 0 0 1, limit lower=-0.9 upper=0.9 effort=12 velocity=4.0
- added joint R_grip_joint: type fixed, parent R_EE, child R_grip_frame, origin xyz=0 0.0375 -0.005 rpy=0 0 0
- added joint R_wrist_ik_joint: type fixed, parent R_wrist_yaw, child R_wrist_ik_frame, origin xyz=0 0 -0.10 rpy=0 0 0
- added joint R_wrist_yaw_joint: type revolute, parent R_elbow, child R_wrist_yaw, origin xyz=0 0 -0.15 rpy=0 0 0, axis 0 0 1, limit lower=-0.9 upper=0.9 effort=12 velocity=4.0
- joint L_EE_joint: axis 0 0 0 -> (none); limit lower=-1.57 upper=1.57 effort=30 velocity=8.5 -> (none); origin xyz=0 0 -0.3 rpy=0 0 0 -> xyz=0 0 -0.15 rpy=0 0 0; parent L_elbow -> L_wrist_yaw
- joint L_shoulder_pitch_joint: origin xyz=-0.0082603 0.16 0.36224 rpy=0.34907 -1.57079632679 0 -> xyz=-0.0082603 0.16 0.36224 rpy=0.34907 0 0
- joint R_EE_joint: axis 0 0 0 -> (none); limit lower=-1.57 upper=1.57 effort=30 velocity=8.5 -> (none); origin xyz=0 0 -0.3 rpy=0 0 0 -> xyz=0 0 -0.15 rpy=0 0 0; parent R_elbow -> R_wrist_yaw
- joint R_shoulder_pitch_joint: origin xyz=-0.0082603 -0.16 0.36224 rpy=-0.34907 -1.57079632679 0 -> xyz=-0.0082603 -0.16 0.36224 rpy=-0.34907 0 0

File: src/Dual_Arm_ROS_Simulation/urdf/dual_arm.xacro (robot description, xacro)
@@ -1,5 +1,9 @@
 <?xml version="1.0" ?>
-<robot name="dual_arm" xmlns:xacro="http://www.ros.org/wiki/xacro">
-<link name="world"/>
+<!-- =================================================================================== -->
+<!-- |    This document was autogenerated by xacro from src/Dual_Arm_ROS_Simulation/urdf/dual_arm.xacro | -->
+<!-- |    EDITING THIS FILE BY HAND IS NOT RECOMMENDED                                 | -->
+<!-- =================================================================================== -->
+<robot name="dual_arm">
+  <link name="world"/>
   <joint name="fixed" type="fixed">
     <parent link="world"/>
@@ -7,743 +11,460 @@
     <origin rpy="0 0 0" xyz="0 0 0.86"/>
   </joint>
-  <link
-    name="Pelvis">
-    <inertial>
-      <origin
-        xyz="-4E-06 1E-05 0.030876"
-        rpy="0 0 0" />
-      <mass
-        value="5.123963" />
-      <inertia
-        ixx="0.051784"
-        ixy="0"
-        ixz="1E-06"
-        iyy="0.01018"
-        iyz="-1E-06"
-        izz="0.055756" />
-    </inertial>
-    <visual>
-      <origin
-        xyz="0 0 0"
-        rpy="0 0 0" />
-      <geometry>
-        <mesh
-          filename="package://dual_arm/meshes/Pelvis.STL" />
-      </geometry>
-      <material
-        name="">
-        <color
-          rgba="0.792156862745098 0.819607843137255 0.933333333333333 1" />
-      </material>
-    </visual>
-    <collision>
-      <origin
-        xyz="0 0 0"
-        rpy="0 0 0" />
-      <geometry>
-        <mesh
-          filename="package://dual_arm/meshes/Pelvis.STL" />
-      </geometry>
-    </collision>
-  </link>
-  <link
-    name="Torso">
-    <inertial>
-      <origin
-        xyz="-0.004339 0 0.216108"
-        rpy="0 0 0" />
-      <mass
-        value="16.636925" />
-      <inertia
-        ixx="0.296782"
-        ixy="-2.9E-05"
-        ixz="-0.0052"
-        iyy="0.232939"
-        iyz="0"
-        izz="0.114483" />
-    </inertial>
-    <visual>
-      <origin
-        xyz="0 0 0"
-        rpy="0 0 0" />
-      <geometry>
-        <mesh
-          filename="package://dual_arm/meshes/Torso.STL" />
-      </geometry>
-      <material
-        name="">
-        <color
-          rgba="0.792156862745098 0.819607843137255 0.933333333333333 1" />
-      </material>
-    </visual>
-    <collision>
-      <origin
-        xyz="0 0 0"
-        rpy="0 0 0" />
-      <geometry>
-        <mesh
-          filename="package://dual_arm/meshes/Torso.STL" />
-      </geometry>
-    </collision>
-  </link>
-  <joint
-    name="Waist_joint"
-    type="revolute">
-    <origin
-      xyz="0 0 0.0825"
-      rpy="0 0 0" />
-    <parent
-      link="Pelvis" />
-    <child
-      link="Torso" />
-    <axis
-      xyz="0 0 1" />
-    <dynamics damping="1"/>
-    <limit
-      lower="-0.87"
-      upper="0.87"
-      effort="100"
-      velocity="13" />
-  </joint>
-  <link
-    name="L_shoulder_pitch">
-    <inertial>
-      <origin
-        xyz="0.010378 0.049076 0"
-        rpy="0 0 0" />
-      <mass
-        value="0.47258" />
-      <inertia
-        ixx="0.000904"
-        ixy="6.4E-05"
-        ixz="0"
-        iyy="0.000955"
-        iyz="0"
-        izz="0.001372" />
-    </inertial>
-    <visual>
-      <origin
-        xyz="0 0 0"
-        rpy="0 0 0" />
-      <geometry>
-        <mesh
-          filename="package://dual_arm/meshes/L_shoulder_pitch.STL" />
-      </geometry>
-      <material
-        name="">
-        <color
-          rgba="0.79216 0.81961 0.93333 1" />
-      </material>
-    </visual>
-    <collision>
-      <origin
-        xyz="0 0 0"
-        rpy="0 0 0" />
-      <geometry>
-        <mesh
-          filename="package://dual_arm/meshes/L_shoulder_pitch.STL" />
-      </geometry>
-    </collision>
-  </link>
-  <joint
-    name="L_shoulder_pitch_joint"
-    type="revolute">
-    <origin
-      xyz="-0.0082603 0.16 0.36224"
-      rpy="0.34907 -1.57079632679 0" />
-    <parent
-      link="Torso" />
-    <child
-      link="L_shoulder_pitch" />
-    <axis
-      xyz="0 1 0" />
-    <dynamics damping="1"/>
-    <limit
-      lower="-3.14"
-      upper="1.05"
-      effort="55"
-      velocity="16" />
-  </joint>
-  <link
-    name="L_shoulder_roll">
-    <inertial>
-      <origin
-        xyz="0.001469 -7E-05 -0.079989"
-        rpy="0 0 0" />
-      <mass
-        value="2.002576" />
-      <inertia
-        ixx="0.020339"
-        ixy="-4E-06"
-        ixz="0.000225"
-        iyy="0.020072"
-        iyz="4.8E-05"
-        izz="0.002315" />
-    </inertial>
-    <visual>
-      <origin
-        xyz="0 0 0"
-        rpy="0 0 0" />
-      <geometry>
-        <mesh
-          filename="package://dual_arm/meshes/L_shoulder_roll.STL" />
-      </geometry>
-      <material
-        name="">
-        <color
-          rgba="0.792156862745098 0.819607843137255 0.933333333333333 1" />
-      </material>
-    </visual>
-    <collision>
-      <origin
-        xyz="0 0 0"
-        rpy="0 0 0" />
-      <geometry>
-        <mesh
-          filename="package://dual_arm/meshes/L_shoulder_roll.STL" />
-      </geometry>
-    </collision>
-  </link>
-  <joint
-    name="L_shoulder_roll_joint"
-    type="revolute">
-    <origin
-      xyz="0.0082603 0.082 0"
-      rpy="-0.261799387799 0 0" />
-    <parent
-      link="L_shoulder_pitch" />
-    <child
-      link="L_shoulder_roll" />
-    <axis
-      xyz="1 0 0" />
-    <dynamics damping="1"/>
-    <limit
-      lower="-0.349"
-      upper="2.62"
-      effort="55"
-      velocity="16" />
-  </joint>
-  <link
-    name="L_shoulder_yaw">
-    <inertial>
-      <origin
-        xyz="4.8E-05 0.00162 -0.045384"
-        rpy="0 0 0" />
-      <mass
-        value="0.608514" />
-      <inertia
-        ixx="0.000608"
-        ixy="0"
-        ixz="0"
-        iyy="0.00049"
-        iyz="-2E-06"
-        izz="0.000483" />
-    </inertial>
-    <visual>
-      <origin
-        xyz="0 0 0"
-        rpy="0 0 0" />
-      <geometry>
-        <mesh
-          filename="package://dual_arm/meshes/L_shoulder_yaw.STL" />
-      </geometry>
-      <material
-        name="">
-        <color
-          rgba="0.792156862745098 0.819607843137255 0.933333333333333 1" />
-      </material>
-    </visual>
-    <collision>
-      <origin
-        xyz="0 0 0"
-        rpy="0 0 0" />
-      <geometry>
-        <mesh
-          filename="package://dual_arm/meshes/L_shoulder_yaw.STL" />
-      </geometry>
-    </collision>
-  </link>
-  <joint
-    name="L_shoulder_yaw_joint"
-    type="revolute">
-    <origin
-      xyz="0 0 -0.2505"
-      rpy="0 0 0" />
-    <parent
-      link="L_shoulder_roll" />
-    <child
-      link="L_shoulder_yaw" />
-    <axis
-      xyz="0 0 1" />
-    <dynamics damping="1"/>
-    <limit
-      lower="-1.57"
-      upper="1.57"
-      effort="30"
-      velocity="8.5" />
-  </joint>
-  <link
-    name="L_elbow">
-    <inertial>
-      <origin
-        xyz="0 -5.2E-05 -0.075944"
-        rpy="0 0 0" />
-      <mass
-        value="0.297153" />
-      <inertia
-        ixx="0.001705"
-        ixy="0"
-        ixz="0"
-        iyy="0.001534"
-        iyz="-1E-06"
-        izz="0.000304" />
-    </inertial>
-    <visual>
-      <origin
-        xyz="0 0 0"
-        rpy="0 0 0" />
-      <geometry>
-        <mesh
-          filename="package://dual_arm/meshes/L_elbow.STL" />
-      </geometry>
-      <material
-        name="">
-        <color
-          rgba="0.792156862745098 0.819607843137255 0.933333333333333 1" />
-      </material>
-    </visual>
-    <collision>
-      <origin
-        xyz="0 0 0"
-        rpy="0 0 0" />
-      <geometry>
-        <mesh
-          filename="package://dual_arm/meshes/L_elbow.STL" />
-      </geometry>
-    </collision>
-  </link>
-  <joint
-    name="L_elbow_joint"
-    type="revolute">
-    <origin
-      xyz="0 0 -0.0545"
-      rpy="0 0 0" />
-    <parent
-      link="L_shoulder_yaw" />
-    <child
-      link="L_elbow" />
-    <axis
-      xyz="0 1 0" />
-    <dynamics damping="1"/>
-    <limit
-      lower="-1.9"
-      upper="1.05"
-      effort="30"
-      velocity="8.5" />
-  </joint>
-  <link
-    name="L_EE">
-    <inertial>
-      <origin
-        xyz="0 0 -0.003514"
-        rpy="0 0 0" />
-      <mass
-        value="0.15" />
-      <inertia
-        ixx="5.5E-05"
-        ixy="0"
-        ixz="0"
-        iyy="5.5E-05"
-        iyz="0"
-        izz="6.4E-05" />
-    </inertial>
-    <visual>
-      <origin
-        xyz="0 0 0"
-        rpy="0 0 0" />
-      <geometry>
-        <mesh
-          filename="package://dual_arm/meshes/L_EE.STL" />
-      </geometry>
-      <material
-        name="">
-        <color
-          rgba="0.298039215686275 0.298039215686275 0.298039215686275 1" />
-      </material>
-    </visual>
-    <collision>
-      <origin
-        xyz="0 0 0"
-        rpy="0 0 0" />
-      <geometry>
-        <mesh
-          filename="package://dual_arm/meshes/L_EE.STL" />
-      </geometry>
-    </collision>
-    <!-- 파지 안정성 보강용 평면 접촉 패드. L_EE.STL은 실측(메시 직접 파싱) 결과 약 6.5x6.5x5.4cm의
-         거의 구형(반경 ~3.25cm)이라 박스 평면과 사실상 점 접촉만 생겨 이송 중 자세가 흔들리기 쉽다.
-         pinocchio FK/IK로 pick 지점(0.45,-0.15,1.20, grasp_offset=0.043) 파지 자세를 직접 풀어보니
-         L_EE 로컬 Y축이 스퀴즈 방향(월드 Y축)의 지배적인 축이라(dot~0.77), 로컬 -Y쪽에 얇은 평면
-         패드를 추가해 둥근 mesh 대신 이 패드가 먼저(mesh 표면보다 1cm 더 튀어나오게) 닿아
-         평면-평면 접촉을 만들도록 한다. 손 마찰(mu=1.2)은 링크 레벨에 지정돼 있어 이 패드에도
-         그대로 적용된다. -->
-    <collision name="L_EE_grip_pad_collision">
-      <origin
-        xyz="0 -0.0375 -0.005"
-        rpy="0 0 0" />
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