Commit message: tune: 손목 컴플라이언스 파지 팔 콜리전 원점 실측 재유도(-0.0375 → 접촉면=EE원점)
배경/문제:
Task 1의 팔 손바닥 콜리전 원점(L=-0.0375, R=+0.0375 in L/R_EE local Y)은
jys 브랜치 수치를 그대로 가져온 추정값이었다. 이 브랜치는 grasp_offset=0.065로
L_EE_joint(=IK 타겟)를 박스 면(중심에서 0.075)보다 10mm 안쪽에 두는데, 여기에
팔 패드가 다시 local -Y로 37.5mm 더 파고들도록 되어 있었다. Gazebo 실측 결과
접촉면(패드 안쪽면)이 박스 면을 약 50mm 관통 → ODE 접촉이 수치적으로 폭발,
좌우 팔이 박스를 밀어내 바닥으로 떨어뜨렸고 L_wrist_yaw가 관절한계(±0.9rad)를
훨씬 넘어 -12rad까지 감기고 F/T가 ±60N으로 진동했다.

검토한 대안과 선택 이유:
(1) grasp_offset을 줄여 관통을 줄이는 방법 - grasp_offset(10mm 압착)은 별도로
튜닝된 값이라 건드리지 않기로 함. (2) 패드 원점을 오프라인 재유도 - 채택.
Pinocchio로 dual_arm.urdf를 로드해 파지 자세 q로 L_EE_joint 프레임을 FK한 결과,
패드 오프셋과 패드 두께가 모두 EE local Y축을 따르므로(투영계수 상쇄) "패드 안쪽면을
EE 원점에 정확히 맞추려면 오프셋 = +두께절반(0.0125)"이라는 방향-무관 결론을 얻음.
이러면 실제 접촉면이 IK 타겟(=grasp_offset 설계값 10mm 관통)과 일치한다.

구현 내용:
urdf/dual_arm.xacro의 L_EE_palm_collision/L_EE_grip_pad_visual 원점 Y를
-0.0375 → +0.0125, R_EE 대응 원점 Y를 +0.0375 → -0.0125로 변경(콜리전/비주얼
4곳). box size(0.090x0.025x0.090), Z(-0.005), X(0)는 유지. xacro로
dual_arm.urdf 재생성.

결과/검증:
Gazebo(gui:=false, 헤드리스 렌더링, target 0.45 0.15 1.2, ArUco 검출
object=[0.467 -0.172 1.216])로 실측. 변경 전: 접촉 즉시 폭발(cf ±60N,
L_wrist=-12rad, 박스 바닥 낙하). 변경 후: 폭발 소멸 — F/T가 유계·정상(cfL≈18.8N
정상 유지, L_wrist≈0.10rad 안정, 감김 없음), 좌팔이 지속 접촉 형성.
단, 파지 자체는 아직 미완: 좌팔이 우팔보다 먼저·세게(18.8N vs 우팔 0N) 접촉하고
잔여토크 tauL_x≈1.56N·m(정렬임계 0.15 초과)로 박스를 world -X로 약 0.3m
밀어내 받침대에서 이탈시킴 → wrist_alignment_ready 미래치, 이송 미도달.
남은 원인(다음 단계): position-only IK가 팔 자세를 구속하지 않아 패드 법선이
world Y(스퀴즈축)와 어긋나(약 -X 0.27, -Z 0.45 성분) 접촉이 면이 아닌 모서리로
발생. 이는 원점(translation)/임계값 튜닝으로 교정 불가 — 자세인지 IK 또는
패드 rpy(타겟 종속) 수준의 후속 작업 필요.

Co-Authored-By: Claude Sonnet 5 <noreply@anthropic.com>

File: urdf/dual_arm.xacro (robot description, xacro)
@@ -396,9 +396,9 @@
          needed 3 rounds of offline recomputation. -->
     <collision name="L_EE_palm_collision">
-      <origin xyz="0 -0.0375 -0.005" rpy="0 0 0" />
+      <origin xyz="0 0.0125 -0.005" rpy="0 0 0" />
       <geometry><box size="0.090 0.025 0.090" /></geometry>
     </collision>
     <visual name="L_EE_grip_pad_visual">
-      <origin xyz="0 -0.0375 -0.005" rpy="0 0 0" />
+      <origin xyz="0 0.0125 -0.005" rpy="0 0 0" />
       <geometry><box size="0.090 0.025 0.090" /></geometry>
       <material name="grip_pad_visual_dark"><color rgba="0.12 0.12 0.12 1" /></material>
@@ -706,9 +706,9 @@
          needed 3 rounds of offline recomputation. -->
     <collision name="R_EE_palm_collision">
-      <origin xyz="0 0.0375 -0.005" rpy="0 0 0" />
+      <origin xyz="0 -0.0125 -0.005" rpy="0 0 0" />
       <geometry><box size="0.090 0.025 0.090" /></geometry>
     </collision>
     <visual name="R_EE_grip_pad_visual">
-      <origin xyz="0 0.0375 -0.005" rpy="0 0 0" />
+      <origin xyz="0 -0.0125 -0.005" rpy="0 0 0" />
       <geometry><box size="0.090 0.025 0.090" /></geometry>
       <material name="grip_pad_visual_dark"><color rgba="0.12 0.12 0.12 1" /></material>
