Commit message: feat: 파지 안정화 및 방향정렬 개선 (jmp-restore)

File: urdf/dual_arm.xacro (robot description, xacro)
@@ -381,4 +381,33 @@
       </geometry>
     </collision>
+    <!-- 파지 안정성 보강용 평면 접촉 패드. L_EE.STL은 실측(메시 직접 파싱) 결과 약 6.5x6.5x5.4cm의
+         거의 구형(반경 ~3.25cm)이라 박스 평면과 사실상 점 접촉만 생겨 이송 중 자세가 흔들리기 쉽다.
+         pinocchio FK/IK로 pick 지점(0.45,-0.15,1.20, grasp_offset=0.043) 파지 자세를 직접 풀어보니
+         L_EE 로컬 Y축이 스퀴즈 방향(월드 Y축)의 지배적인 축이라(dot~0.77), 로컬 -Y쪽에 얇은 평면
+         패드를 추가해 둥근 mesh 대신 이 패드가 먼저(mesh 표면보다 1cm 더 튀어나오게) 닿아
+         평면-평면 접촉을 만들도록 한다. 손 마찰(mu=1.2)은 링크 레벨에 지정돼 있어 이 패드에도
+         그대로 적용된다. -->
+    <collision name="L_EE_grip_pad_collision">
+      <origin
+        xyz="0 -0.0375 -0.005"
+        rpy="0 0 0" />
+      <geometry>
+        <box size="0.04 0.01 0.04" />
+      </geometry>
+    </collision>
+    <!-- L자형 턱(lip): 패드는 마찰(μN)에만 의존하므로 접촉 예산 자체는 늘려주지 않는다. 물체
+         아래 모서리를 기하학적으로 받칠 수 있도록 패드 아래쪽에 1cm 턱을 추가한다.
+         로컬축 매핑(위 pick 자세 FK 실측): 로컬 +X가 월드 +Z(수직, dot~0.97)와 거의 나란하고
+         로컬 Y가 스퀴즈 방향이다 - 그래서 "아래"는 로컬 -X, "물체 쪽으로 더 뻗기"는 로컬 -Y다.
+         패드 바닥(로컬 x=-0.02) 바로 아래, 패드 바깥면(로컬 y=-0.0425)보다 1cm 더 뻗어나가게
+         배치해서 물체가 미끄러져 내려오면 이 턱에 걸리도록 한다. -->
+    <collision name="L_EE_grip_lip_collision">
+      <origin
+        xyz="-0.025 -0.0475 -0.005"
+        rpy="0 0 0" />
+      <geometry>
+        <box size="0.01 0.01 0.04" />
+      </geometry>
+    </collision>
   </link>
   <joint
@@ -674,4 +703,26 @@
         <mesh
           filename="package://dual_arm/meshes/R_EE.STL" />
+      </geometry>
+    </collision>
+    <!-- 파지 안정성 보강용 평면 접촉 패드 (L_EE 쪽 설명 참고, mesh 반경 ~3.25cm). R_EE 로컬 Y축은
+         FK/IK 실측상 스퀴즈 방향(월드 Y축)과 거의 완벽히 정렬돼(dot~0.99) L_EE보다 정렬이 더
+         좋다. 로컬 +Y쪽에 배치, mesh 표면보다 1cm 더 튀어나오게 해서 이 패드가 먼저 닿는다. -->
+    <collision name="R_EE_grip_pad_collision">
+      <origin
+        xyz="0 0.0375 -0.005"
+        rpy="0 0 0" />
+      <geometry>
+        <box size="0.04 0.01 0.04" />
+      </geometry>
+    </collision>
+    <!-- L자형 턱(lip) - L_EE 쪽 설명/축 매핑 참고 (R도 로컬 +X가 월드 +Z와 dot~0.97로 거의
+         나란함). 패드 바닥(로컬 x=-0.02) 아래, 패드 바깥면(로컬 y=0.0425)보다 1cm 더 뻗어나가게
+         배치. -->
+    <collision name="R_EE_grip_lip_collision">
+      <origin
+        xyz="-0.025 0.0475 -0.005"
+        rpy="0 0 0" />
+      <geometry>
+        <box size="0.01 0.01 0.04" />
       </geometry>
     </collision>
@@ -857,4 +908,31 @@
     </sensor>
   </gazebo>
+  <!-- L_EE_joint/R_EE_joint는 fixed 조인트라 URDF->SDF 변환 시 부모 링크(L_elbow/R_elbow)로
+       lumping(축약)될 수 있다. lumping되면 조인트 자체가 사라져서 force_torque 피드백을 못 얻으므로
+       명시적으로 lumping을 막고 조인트 피드백 계산을 켠다. -->
+  <gazebo reference="L_EE_joint">
+    <disableFixedJointLumping>true</disableFixedJointLumping>
+    <provideFeedback>true</provideFeedback>
+  </gazebo>
+  <gazebo reference="R_EE_joint">
+    <disableFixedJointLumping>true</disableFixedJointLumping>
+    <provideFeedback>true</provideFeedback>
+  </gazebo>
+  <!-- gazebo_ros_ft_sensor: L_EE_joint/R_EE_joint에 걸리는 반력을 각각
+       /dual_arm/left_ft_sensor, /dual_arm/right_ft_sensor (geometry_msgs/WrenchStamped)로 발행. -->
+  <gazebo>
+    <plugin name="l_ee_ft_sensor" filename="libgazebo_ros_ft_sensor.so">
+      <updateRate>100.0</updateRate>
+      <topicName>/dual_arm/left_ft_sensor</topicName>
+      <jointName>L_EE_joint</jointName>
+    </plugin>
+  </gazebo>
+  <gazebo>
+    <plugin name="r_ee_ft_sensor" filename="libgazebo_ros_ft_sensor.so">
+      <updateRate>100.0</updateRate>
+      <topicName>/dual_arm/right_ft_sensor</topicName>
+      <jointName>R_EE_joint</jointName>
+    </plugin>
+  </gazebo>
   <link
     name="L_hip">

Commit message: feat: 그립 패드를 사각+L자턱 조합에서 원형 평면 패드로 교체
배경/문제:
기존 그립 패드는 손 mesh(L_EE/R_EE, 거의 구형) 표면 위에 사각 평면 패드(4x1x4cm box)와
그 아래 L자형 턱(1x1x4cm box)을 붙여, 패드는 면 접촉을, 턱은 물체 아래 모서리를 기하학적으로
받치는 역할을 나누어 맡고 있었다. 실제 Gazebo 시각화 결과 패드/턱 모두 <collision>만 있고
<visual>이 없어 눈에 전혀 보이지 않았고(사용자 지적), 정면에서 보면 접촉 형상 자체도 힘이
잘 전달될 구조로 보이지 않았다.

검토한 대안과 선택 이유:
1) L자 턱을 그대로 유지하고 visual만 추가 - 형상 자체의 문제(마찰(μN)에만 의존, 접촉 예산이
   늘지 않음)는 그대로 남아 기각.
2) 사각 패드+턱 조합을 원형 평면 패드(cylinder) 하나로 통합 - 턱이 제공하던 "모서리를
   기하학적으로 거는" 기능은 없어지고 순수 마찰 접촉면이 되지만, 사용자와 확인 후 이 방향으로
   진행하기로 함(순수 마찰 기반, 반지름/두께는 이후 실험으로 튜닝).

구현 내용:
- L_EE_grip_pad_collision + L_EE_grip_lip_collision -> L_EE_grip_disc_visual/collision
  하나로 통합 (R_EE도 동일). geometry는 box에서 cylinder(radius=0.03m, length=0.01m)로 변경,
  주황색(rgba 1.0 0.5 0.0 1) 머티리얼 추가.
- rpy는 fk_pad_calc.cpp(일회성 도구, 커밋 안 함)로 재계산: main.cpp의 실제 vision pick
  파이프라인(base_seed=0 스폰 상태 -> segment 1 start->standoff -> segment 1b standoff->접촉,
  동일한 SolveIK_Position/CartesianLineTrajectory/grasp_offset=0.040/STANDOFF_Y=0.15/v_des)을
  처음부터 그대로 재현해서 실제 파지 순간 L_EE/R_EE의 world 자세를 구한 뒤, 원판 법선(로컬 Z축)이
  파지 시점 물체 옆면 법선(월드 Y축)과 정확히 평행해지도록 역산했다.
- origin xyz는 사용자 요청에 따라 파지 시점 자세 기준 월드 Z축으로 총 1.5cm(왼손)/0.5cm(오른손)
  올렸다 - 각 손의 실제 파지 자세 회전행렬로 월드 Z 이동량을 로컬 좌표로 역변환해서 반영.

결과/검증:
매 단계 `rosrun xacro xacro --inorder`로 문법 검증(exit 0) 후 catkin_make 빌드 성공을 확인했다.
fk_pad_calc.cpp 계산 결과 원판 법선과 물체 옆면 법선의 dot product=1.0(완벽 정렬)으로 검증했다.
Gazebo에서 육안으로 확인한 결과 파지가 거의 평행하게 이루어지는 것을 확인했으나, 정면에서 보면
힘이 제대로 전달되는 것처럼 보이지 않는다는 관찰이 있어(이후 F/T 센서 실측으로 이어짐), 형상/위치
자체는 이 커밋으로 일단락하고 힘 전달 문제는 별도로 진단 중이다.

File: urdf/dual_arm.xacro (robot description, xacro)
@@ -392,22 +392,28 @@
          (계산: fk_debug.cpp, 일회성 도구, 커밋 안 함). 위치(xyz)는 그대로 두고 방향만 보정 -
          정확한 돌출거리 재튜닝(전체 손 형상 재설계, P2)은 이후 과제로 보류. -->
-    <collision name="L_EE_grip_pad_collision">
-      <origin
-        xyz="0 -0.0375 -0.005"
-        rpy="0.699086 0.041596 -0.114007" />
-      <geometry>
-        <box size="0.04 0.01 0.04" />
-      </geometry>
-    </collision>
-    <!-- L자형 턱(lip): 패드는 마찰(μN)에만 의존하므로 접촉 예산 자체는 늘려주지 않는다. 물체
-         아래 모서리를 기하학적으로 받칠 수 있도록 패드 아래쪽에 1cm 턱을 추가한다. 패드와 동일한
-         보정 rpy를 적용해 패드-턱의 상대 배치(로컬 -X 아래, 로컬 -Y 바깥쪽 1cm 더 뻗음)를 유지한다 -
-         위 패드 주석의 fk_debug 보정과 동일 근거. -->
-    <collision name="L_EE_grip_lip_collision">
-      <origin
-        xyz="-0.025 -0.0475 -0.005"
-        rpy="0.699086 0.041596 -0.114007" />
-      <geometry>
-        <box size="0.01 0.01 0.04" />
+    <!-- 원형 접촉 패드: 기존 사각 패드(box)+L자형 턱 조합을 하나의 평평한 원판(cylinder)으로 교체.
+         rpy는 실제 vision pick 파이프라인(base_seed=0 스폰 상태 -> segment 1 standoff -> segment 1b
+         접촉, main.cpp와 동일한 SolveIK_Position/CartesianLineTrajectory/grasp_offset=0.040/
+         STANDOFF_Y=0.15/v_des를 그대로 재현)을 처음부터 다시 풀어서, 실제 파지 순간 L_EE 프레임의
+         world 자세를 구한 뒤, 원판 법선(로컬 Z축)이 파지 시점 물체 옆면 법선(월드 Y축)과 정확히
+         평행해지는 방향으로 역산했다 (계산: fk_pad_calc.cpp, 일회성 도구, 커밋 안 함, dot=1.0 검증).
+         위치(origin xyz)는 기존 패드 자리를 그대로 재사용 - mesh 표면 돌출거리 재튜닝은 보류. -->
+    <visual name="L_EE_grip_disc_visual">
+      <origin
+        xyz="0.009786 -0.030398 0.003877"
+        rpy="1.224122 -0.000000 -2.245407" />
+      <geometry>
+        <cylinder radius="0.03" length="0.01" />
+      </geometry>
+      <material name="grip_pad_orange">
+        <color rgba="1.0 0.5 0.0 1" />
+      </material>
+    </visual>
+    <collision name="L_EE_grip_disc_collision">
+      <origin
+        xyz="0.009786 -0.030398 0.003877"
+        rpy="1.224122 -0.000000 -2.245407" />
+      <geometry>
+        <cylinder radius="0.03" length="0.01" />
       </geometry>
     </collision>
@@ -713,19 +719,23 @@
          무시할 수준은 아니다. L_EE와 동일한 방식으로 rpy를 target_local_dir(=R_EE^T*worldY)에
          맞춰 보정한다 (계산: fk_debug.cpp, 일회성 도구, 커밋 안 함). -->
-    <collision name="R_EE_grip_pad_collision">
-      <origin
-        xyz="0 0.0375 -0.005"
-        rpy="-0.206731 -0.022471 -0.215784" />
-      <geometry>
-        <box size="0.04 0.01 0.04" />
-      </geometry>
-    </collision>
-    <!-- L자형 턱(lip) - L_EE 쪽 설명 참고. 패드와 동일한 보정 rpy를 적용해 상대 배치를 유지한다. -->
-    <collision name="R_EE_grip_lip_collision">
-      <origin
-        xyz="-0.025 0.0475 -0.005"
-        rpy="-0.206731 -0.022471 -0.215784" />
-      <geometry>
-        <box size="0.01 0.01 0.04" />
+    <!-- 원형 접촉 패드 - L_EE 쪽 설명 참고. 동일한 방식(fk_pad_calc.cpp로 파지 파이프라인 처음부터
+         재현)으로 rpy 재계산, dot=1.0 검증. -->
+    <visual name="R_EE_grip_disc_visual">
+      <origin
+        xyz="0.003329 0.035647 -0.001762"
+        rpy="1.441584 -0.000000 2.744360" />
+      <geometry>
+        <cylinder radius="0.03" length="0.01" />
+      </geometry>
+      <material name="grip_pad_orange">
+        <color rgba="1.0 0.5 0.0 1" />
+      </material>
+    </visual>
+    <collision name="R_EE_grip_disc_collision">
+      <origin
+        xyz="0.003329 0.035647 -0.001762"
+        rpy="1.441584 -0.000000 2.744360" />
+      <geometry>
+        <cylinder radius="0.03" length="0.01" />
       </geometry>
     </collision>

Commit message: tune: 그립 패드 접촉 강성/댐핑을 Gazebo ODE 기본값에서 낮춰 재설정
배경/문제:
F/T 센서 실측(Gazebo에서 vision pick 1회 실행, left/right_ft_sensor 로깅)으로 확인한 결과,
grasp_to_place(들어올려서 이송) 구간 평균 |Fy|가 목표 스퀴즈력(ADMITTANCE_FD_Y=10N) 대비
왼손 22%, 오른손 42%에 그쳤고 부호가 계속 뒤집히며 진동했다(왼손 -15~+14N, 오른손 -25~+16N) -
꾸준한 압착이 아니라 접촉이 붙었다 떨어졌다 하는 모습이었다. 원인 조사 중 이 프로젝트의 URDF/SDF
어디에도 <contact> kp/kd가 명시된 적이 없어, 설치된 sdformat9(Gazebo 11) 스키마 기본값
kp=1e12(사실상 강체), kd=1.0을 그대로 쓰고 있었던 것을 확인했다. kp가 극단적으로 높으면 접촉
순간 임펄스성 반발력이 커져 접촉/이탈이 반복되기 쉽다는 가설을 세웠다.

검토한 대안과 선택 이유:
접촉 강성/댐핑을 낮춰 접촉을 더 부드럽게(덜 튀게) 만드는 방향으로, kp를 1e12에서 1e5로,
kd를 1.0에서 100.0으로 설정했다(사용자 제공 값). minDepth=0.003(약간의 침투 허용으로 접촉
안정성 향상), maxVel=0.0(접촉 보정 최대속도 제한 해제)도 함께 적용했다. mu1/mu2=1.2는 기존
박스 쪽 마찰계수와 동일하게 맞춰 명시적으로 설정 - 기존에는 손/패드 쪽에 마찰계수 자체가
설정되어 있지 않아 어떤 조합 법칙이 적용되는지 불명확했던 문제도 같이 해소한다.

구현 내용:
dual_arm.xacro의 L_EE_joint/R_EE_joint ft_sensor 블록 사이에 <gazebo reference="L_EE">,
<gazebo reference="R_EE"> 블록을 추가. urdf2sdf 변환 시 이 두 링크(그립 원판이 고정 자식으로
붙어있는 링크)의 모든 collision(mesh + 원판)에 반영된다.

결과/검증:
`rosrun xacro xacro --inorder`로 문법 검증(exit 0) 및 생성된 URDF에 태그가 정상 포함되는 것을
확인했고, catkin_make 빌드 성공을 확인했다. 실제 Gazebo 재실행 + F/T 재측정을 통한 접촉 임펄스
감소 여부 검증은 다음 세션에서 진행 예정.

File: urdf/dual_arm.xacro (robot description, xacro)
@@ -932,4 +932,24 @@
     <provideFeedback>true</provideFeedback>
   </gazebo>
+  <!-- 왼쪽/오른쪽 패드 접촉 특성 변경: 기본 kp=1e12(사실상 강체)를 낮춰 접촉 시 임펄스성 반발력을
+       줄이고, minDepth로 약간의 침투를 허용해 접촉 안정성을 높인다. L_EE/R_EE 링크(그립 원판이
+       고정 자식으로 붙어있는 링크)에 적용 - urdf2sdf 변환 시 이 링크의 모든 <collision>(mesh +
+       원판) 표면에 반영된다. -->
+  <gazebo reference="L_EE">
+    <mu1>1.2</mu1>
+    <mu2>1.2</mu2>
+    <kp>100000.0</kp>
+    <kd>100.0</kd>
+    <minDepth>0.003</minDepth>
+    <maxVel>0.0</maxVel>
+  </gazebo>
+  <gazebo reference="R_EE">
+    <mu1>1.2</mu1>
+    <mu2>1.2</mu2>
+    <kp>100000.0</kp>
+    <kd>100.0</kd>
+    <minDepth>0.003</minDepth>
+    <maxVel>0.0</maxVel>
+  </gazebo>
   <!-- gazebo_ros_ft_sensor: L_EE_joint/R_EE_joint에 걸리는 반력을 각각
        /dual_arm/left_ft_sensor, /dual_arm/right_ft_sensor (geometry_msgs/WrenchStamped)로 발행. -->

Commit message: feat: 손목 yaw 관절용 트랜스미션 및 컨트롤러(joint12/13) 추가
배경/문제:
Task 1에서 추가한 L_wrist_yaw_joint/R_wrist_yaw_joint는 트랜스미션과
ros_control 컨트롤러 설정이 없으면 액추에이터가 없는 관절이라 Gazebo에서
전혀 움직일 수 없다. Task 4(C++ 쪽에서 이 관절을 커맨드)의 전제 조건.

검토한 대안과 선택 이유:
기존 joint1~11 컨트롤러 이름/번호를 재사용하는 대신 joint12/13으로 끝에
추가 - 기존 컨트롤러를 재번호 매기면 이 이름들을 참조하는 다른 launch
파일/설정이 깨질 위험이 있어 surgical하게 append만 함.

트랜스미션 mechanicalReduction 값과 관련해 계획서(brief)의 서술과 실제
파일 내용이 다름을 발견해 계획서 대신 실제 파일을 따랐다: brief는
"Waist_joint=50, L_elbow_joint 같은 팔 관절=1"처럼 관절별로 값이 다르다고
서술했지만, 실제로는 섹션별로 값이 결정된다 - Position Control 섹션
(tran1~11, 전체가 XML 주석으로 비활성화된 상태)은 Waist_joint 포함 전부
50, Effort Control 섹션(활성 상태, 실제로 launch/dual_arm_control.launch
스포너가 로드하는 쪽)은 Waist_joint 포함 전부 1. 같은 섹션 안에서
L_elbow_joint와 Waist_joint가 다른 reduction을 쓰는 경우는 없었다. 따라서
새 손목 관절도 "그 섹션에 이미 있는 값"을 따라 Position 섹션엔 50,
Effort 섹션엔 1을 사용 - 실질적으로 동작하는 Effort 섹션 값은 brief가
원한 값(1)과 정확히 일치하고, 비활성 상태인 Position 섹션 값(50)은
현재 아무 런타임 영향이 없다.

PID는 jys의 Kp=40/Kd=8(다른 관절 대비 훨씬 무른 값, 컴플라이언스 목적)을
그대로 가져옴 - Task 3의 C++ Kp[DoF]/Kd[DoF] 배열과 반드시 동일하게
유지해야 함.

구현 내용:
urdf/dual_arm.xacro에 L_wrist_yaw_joint/R_wrist_yaw_joint용 tran_L_wrist/
tran_R_wrist SimpleTransmission을 Position/Effort 두 섹션에 각각 추가
(actuator 이름도 motor_L_wrist/motor_R_wrist로 기존 팔 관절과 같은 재사용
패턴). urdf/dual_arm.urdf는 xacro로 재생성해 소스와 동기화. 두 yaml
설정 파일 각각에 joint12/13_..._controller 추가(p:40, i:0, d:8), 기존
joint1~11 블록은 손대지 않음.

Step 3 확인 결과 brief가 지목한 launch/gazebo.launch 자체에는 스포너가
없고, 이 파일이 include하는 launch/dual_arm_control.launch에 실제
controller_manager/spawner 노드 2개(Position용 - 주석 처리로 비활성,
Effort용 - 활성)가 있었다. 둘 다 컨트롤러 이름을 args에 명시적으로
나열하는 방식이라 와일드카드가 아니었음 - 활성 상태인 Effort 스포너
args에 joint12_effort_controller/joint13_effort_controller를 추가했고
(이게 없으면 yaml에 컨트롤러가 정의돼도 실제로 스폰되지 않음), 비활성
Position 스포너에도 대칭성을 위해 joint12/13_position_controller를
같이 추가했다(현재는 주석 블록이라 런타임 영향 없음).

결과/검증:
python yaml.safe_load로 두 설정 파일 다 14개 컨트롤러 키(joint_state +
joint1~13)를 갖고 있음을 확인. xml.dom.minidom으로 xacro가 여전히
well-formed XML임을 확인. xacro urdf/dual_arm.xacro > urdf/dual_arm.urdf로
재생성 후 pinocchio buildModelFromUrdf로 로드해 nq=nv=13(Task 1과 동일)
확인 - 트랜스미션 추가가 URDF 파싱이나 기구학 모델에 영향을 주지 않음을
검증. Gazebo 실제 스폰 검증은 Task 3(IK가 이 관절을 인식하도록 C++ 코드
확장, DoF=11→13) 이후로 미룸.

File: urdf/dual_arm.xacro (robot description, xacro)
@@ -1634,4 +1634,24 @@
       <mechanicalReduction>50</mechanicalReduction>
     </actuator>
+  </transmission>
+  <transmission name="tran_L_wrist">
+    <type>transmission_interface/SimpleTransmission</type>
+    <joint name="L_wrist_yaw_joint">
+      <hardwareInterface>hardware_interface/PositionJointInterface</hardwareInterface>
+    </joint>
+    <actuator name="motor_L_wrist">
+      <hardwareInterface>hardware_interface/PositionJointInterface</hardwareInterface>
+      <mechanicalReduction>50</mechanicalReduction>
+    </actuator>
+  </transmission>
+  <transmission name="tran_R_wrist">
+    <type>transmission_interface/SimpleTransmission</type>
+    <joint name="R_wrist_yaw_joint">
+      <hardwareInterface>hardware_interface/PositionJointInterface</hardwareInterface>
+    </joint>
+    <actuator name="motor_R_wrist">
+      <hardwareInterface>hardware_interface/PositionJointInterface</hardwareInterface>
+      <mechanicalReduction>50</mechanicalReduction>
+    </actuator>
   </transmission> -->
   <!-- Effort Control -->
@@ -1742,4 +1762,24 @@
     </joint>
     <actuator name="motor11">
+      <hardwareInterface>hardware_interface/EffortJointInterface</hardwareInterface>
+      <mechanicalReduction>1</mechanicalReduction>
+    </actuator>
+  </transmission>
+  <transmission name="tran_L_wrist">
+    <type>transmission_interface/SimpleTransmission</type>
+    <joint name="L_wrist_yaw_joint">
+      <hardwareInterface>hardware_interface/EffortJointInterface</hardwareInterface>
+    </joint>
+    <actuator name="motor_L_wrist">
+      <hardwareInterface>hardware_interface/EffortJointInterface</hardwareInterface>
+      <mechanicalReduction>1</mechanicalReduction>
+    </actuator>
+  </transmission>
+  <transmission name="tran_R_wrist">
+    <type>transmission_interface/SimpleTransmission</type>
+    <joint name="R_wrist_yaw_joint">
+      <hardwareInterface>hardware_interface/EffortJointInterface</hardwareInterface>
+    </joint>
+    <actuator name="motor_R_wrist">
       <hardwareInterface>hardware_interface/EffortJointInterface</hardwareInterface>
       <mechanicalReduction>1</mechanicalReduction>

Commit message: feat: extend effort control stack to 15DoF

File: urdf/dual_arm.xacro (robot description, xacro)
@@ -1866,68 +1866,88 @@
   <transmission name="tran7">
     <type>transmission_interface/SimpleTransmission</type>
+    <joint name="L_wrist_pitch_joint">
+      <hardwareInterface>hardware_interface/EffortJointInterface</hardwareInterface>
+    </joint>
+    <actuator name="motor7">
+      <hardwareInterface>hardware_interface/EffortJointInterface</hardwareInterface>
+      <mechanicalReduction>1</mechanicalReduction>
+    </actuator>
+  </transmission>
+  <transmission name="tran8">
+    <type>transmission_interface/SimpleTransmission</type>
     <joint name="R_shoulder_pitch_joint">
       <hardwareInterface>hardware_interface/EffortJointInterface</hardwareInterface>
     </joint>
-    <actuator name="motor7">
+    <actuator name="motor8">
       <hardwareInterface>hardware_interface/EffortJointInterface</hardwareInterface>
       <mechanicalReduction>1</mechanicalReduction>
     </actuator>
   </transmission>
-  <transmission name="tran8">
+  <transmission name="tran9">
     <type>transmission_interface/SimpleTransmission</type>
     <joint name="R_shoulder_roll_joint">
       <hardwareInterface>hardware_interface/EffortJointInterface</hardwareInterface>
     </joint>
-    <actuator name="motor8">
+    <actuator name="motor9">
       <hardwareInterface>hardware_interface/EffortJointInterface</hardwareInterface>
       <mechanicalReduction>1</mechanicalReduction>
     </actuator>
   </transmission>
-  <transmission name="tran9">
+  <transmission name="tran10">
     <type>transmission_interface/SimpleTransmission</type>
     <joint name="R_shoulder_yaw_joint">
       <hardwareInterface>hardware_interface/EffortJointInterface</hardwareInterface>
     </joint>
-    <actuator name="motor9">
+    <actuator name="motor10">
       <hardwareInterface>hardware_interface/EffortJointInterface</hardwareInterface>
       <mechanicalReduction>1</mechanicalReduction>
     </actuator>
   </transmission>
-  <transmission name="tran10">
+  <transmission name="tran11">
     <type>transmission_interface/SimpleTransmission</type>
     <joint name="R_elbow_joint">
       <hardwareInterface>hardware_interface/EffortJointInterface</hardwareInterface>
     </joint>
-    <actuator name="motor10">
+    <actuator name="motor11">
       <hardwareInterface>hardware_interface/EffortJointInterface</hardwareInterface>
       <mechanicalReduction>1</mechanicalReduction>
     </actuator>
   </transmission>
-  <transmission name="tran11">
+  <transmission name="tran12">
     <type>transmission_interface/SimpleTransmission</type>
     <joint name="R_wrist_yaw_joint">
       <hardwareInterface>hardware_interface/EffortJointInterface</hardwareInterface>
     </joint>
-    <actuator name="motor11">
+    <actuator name="motor12">
       <hardwareInterface>hardware_interface/EffortJointInterface</hardwareInterface>
       <mechanicalReduction>1</mechanicalReduction>
     </actuator>
   </transmission>
-  <transmission name="tran12">
+  <transmission name="tran13">
+    <type>transmission_interface/SimpleTransmission</type>
+    <joint name="R_wrist_pitch_joint">
+      <hardwareInterface>hardware_interface/EffortJointInterface</hardwareInterface>
+    </joint>
+    <actuator name="motor13">
+      <hardwareInterface>hardware_interface/EffortJointInterface</hardwareInterface>
+      <mechanicalReduction>1</mechanicalReduction>
+    </actuator>
+  </transmission>
+  <transmission name="tran14">
     <type>transmission_interface/SimpleTransmission</type>
     <joint name="Head_yaw_joint">
       <hardwareInterface>hardware_interface/EffortJointInterface</hardwareInterface>
     </joint>
-    <actuator name="motor12">
+    <actuator name="motor14">
       <hardwareInterface>hardware_interface/EffortJointInterface</hardwareInterface>
       <mechanicalReduction>1</mechanicalReduction>
     </actuator>
   </transmission>
-  <transmission name="tran13">
+  <transmission name="tran15">
     <type>transmission_interface/SimpleTransmission</type>
     <joint name="Head_pitch_joint">
       <hardwareInterface>hardware_interface/EffortJointInterface</hardwareInterface>
     </joint>
-    <actuator name="motor13">
+    <actuator name="motor15">
       <hardwareInterface>hardware_interface/EffortJointInterface</hardwareInterface>
       <mechanicalReduction>1</mechanicalReduction>

Commit message: feat: 손목 pitch 관절(joint14/15)용 트랜스미션 및 컨트롤러 추가
배경/문제:
Task 1(45f6dcc)에서 URDF에 L_wrist_pitch_joint/R_wrist_pitch_joint를 추가했으나,
트랜스미션과 ros_control 컨트롤러가 없으면 액추에이터가 없는 관절이라 Gazebo에서
전혀 움직일 수 없다. 853b0bc가 wrist_yaw(joint12/13)에 적용한 것과 동일한 배선을
새 pitch 관절(joint14/15)에도 반복해야 한다.

검토한 대안과 선택 이유:
853b0bc가 이미 확립한 패턴을 그대로 따름: 트랜스미션 mechanicalReduction은
관절이 아니라 섹션 단위로 결정되므로(비활성 Position 섹션=50, 실제 launch가
로드하는 활성 Effort 섹션=1) 계획서의 "관절별 값" 가정 대신 각 섹션에 이미
존재하는 값을 그대로 따랐다. yaml PID는 wrist_yaw와 동일한 p:40/i:0/d:8(컴플라이언스
목적의 무른 게인)을 그대로 사용 - Task 3의 C++ Kp/Kd 배열과 반드시 동일해야 함.
joint1~13은 번호를 그대로 두고 joint14/15만 끝에 append.

구현 내용:
urdf/dual_arm.xacro에 L/R_wrist_pitch_joint용 SimpleTransmission을 Position/Effort
두 섹션에 각각 추가(tran_L_wrist_pitch/tran_R_wrist_pitch), xacro→urdf 재생성.
config/dual_arm_positioncontrol.yaml, dual_arm_effortcontrol.yaml에 joint14/15
컨트롤러 append(p:40, i:0, d:8), 기존 joint1~13 블록은 변경 없음.
launch/dual_arm_control.launch의 두 스포너(Position-비활성/Effort-활성) args에
joint14/15 컨트롤러 이름을 853b0bc와 동일한 패턴으로(두 섹션 모두) 추가 - 실제
로드되는 건 활성 Effort 스포너뿐이지만, 853b0bc가 joint12/13을 비활성 Position
스포너 args에도 같이 넣어둔 기존 패턴을 그대로 따랐다.

결과/검증:
python yaml.safe_load로 두 설정 파일 다 16개 컨트롤러 키(joint_state +
joint1~15) 확인. xml.dom.minidom으로 xacro가 well-formed XML임을 확인.
xacro로 urdf 재생성 성공. Gazebo 실제 스폰 검증은 Task 3(IK가 이 관절을
인식하도록 C++ 코드 확장, DoF 13→15) 이후로 미룸.

File: urdf/dual_arm.xacro (robot description, xacro)
@@ -1684,4 +1684,24 @@
       <mechanicalReduction>50</mechanicalReduction>
     </actuator>
+  </transmission>
+  <transmission name="tran_L_wrist_pitch">
+    <type>transmission_interface/SimpleTransmission</type>
+    <joint name="L_wrist_pitch_joint">
+      <hardwareInterface>hardware_interface/PositionJointInterface</hardwareInterface>
+    </joint>
+    <actuator name="motor_L_wrist_pitch">
+      <hardwareInterface>hardware_interface/PositionJointInterface</hardwareInterface>
+      <mechanicalReduction>50</mechanicalReduction>
+    </actuator>
+  </transmission>
+  <transmission name="tran_R_wrist_pitch">
+    <type>transmission_interface/SimpleTransmission</type>
+    <joint name="R_wrist_pitch_joint">
+      <hardwareInterface>hardware_interface/PositionJointInterface</hardwareInterface>
+    </joint>
+    <actuator name="motor_R_wrist_pitch">
+      <hardwareInterface>hardware_interface/PositionJointInterface</hardwareInterface>
+      <mechanicalReduction>50</mechanicalReduction>
+    </actuator>
   </transmission> -->
   <!-- Effort Control -->
@@ -1812,4 +1832,24 @@
     </joint>
     <actuator name="motor_R_wrist">
+      <hardwareInterface>hardware_interface/EffortJointInterface</hardwareInterface>
+      <mechanicalReduction>1</mechanicalReduction>
+    </actuator>
+  </transmission>
+  <transmission name="tran_L_wrist_pitch">
+    <type>transmission_interface/SimpleTransmission</type>
+    <joint name="L_wrist_pitch_joint">
+      <hardwareInterface>hardware_interface/EffortJointInterface</hardwareInterface>
+    </joint>
+    <actuator name="motor_L_wrist_pitch">
+      <hardwareInterface>hardware_interface/EffortJointInterface</hardwareInterface>
+      <mechanicalReduction>1</mechanicalReduction>
+    </actuator>
+  </transmission>
+  <transmission name="tran_R_wrist_pitch">
+    <type>transmission_interface/SimpleTransmission</type>
+    <joint name="R_wrist_pitch_joint">
+      <hardwareInterface>hardware_interface/EffortJointInterface</hardwareInterface>
+    </joint>
+    <actuator name="motor_R_wrist_pitch">
       <hardwareInterface>hardware_interface/EffortJointInterface</hardwareInterface>
       <mechanicalReduction>1</mechanicalReduction>
