Commit message: feat: 카메라 마운트, ArUco 인식, 양팔 동시 파지 궤적, vision pick 모드 구현

File: urdf/dual_arm.urdf (robot description, URDF)
Before this commit: robot dual_arm, 25 links, 24 joints
Links:
- added link Head_camera_link, mass 0.05; visual sphere radius=0.02
- added link Head_camera_link_optical
Joints:
- added joint Head_camera_joint: type fixed, parent Head, child Head_camera_link, origin xyz=0.05 0 0.145 rpy=0 0 0
- added joint Head_camera_optical_joint: type fixed, parent Head_camera_link, child Head_camera_link_optical, origin xyz=0 0 0 rpy=-1.5707963 0 -1.5707963

File: urdf/dual_arm.xacro (robot description, xacro)
@@ -773,4 +773,88 @@
       velocity="8.5" />
   </joint>
+  <!-- Head-mounted RGB-D camera -->
+  <link
+    name="Head_camera_link">
+    <inertial>
+      <origin xyz="0 0 0" rpy="0 0 0" />
+      <mass value="0.05" />
+      <inertia ixx="1E-05" ixy="0" ixz="0" iyy="1E-05" iyz="0" izz="1E-05" />
+    </inertial>
+    <visual>
+      <origin xyz="0 0 0" rpy="0 0 0" />
+      <geometry>
+        <sphere radius="0.02" />
+      </geometry>
+      <material name="camera_marker_red">
+        <color rgba="1 0 0 1" />
+      </material>
+    </visual>
+  </link>
+  <joint
+    name="Head_camera_joint"
+    type="fixed">
+    <origin
+      xyz="0.05 0 0.145"
+      rpy="0 0 0" />
+    <parent
+      link="Head" />
+    <child
+      link="Head_camera_link" />
+  </joint>
+  <!-- Optical frame: rotates to ROS REP-103 camera-optical convention (x-right, y-down, z-forward) -->
+  <link name="Head_camera_link_optical" />
+  <joint
+    name="Head_camera_optical_joint"
+    type="fixed">
+    <origin
+      xyz="0 0 0"
+      rpy="-1.5707963 0 -1.5707963" />
+    <parent
+      link="Head_camera_link" />
+    <child
+      link="Head_camera_link_optical" />
+  </joint>
+  <gazebo reference="Head_camera_link">
+    <sensor type="depth" name="head_camera">
+      <update_rate>20</update_rate>
+      <camera>
+        <horizontal_fov>1.047</horizontal_fov>
+        <image>
+          <width>640</width>
+          <height>480</height>
+          <format>R8G8B8</format>
+        </image>
+        <clip>
+          <near>0.05</near>
+          <far>10.0</far>
+        </clip>
+      </camera>
+      <plugin name="head_camera_controller" filename="libgazebo_ros_openni_kinect.so">
+        <baseline>0.1</baseline>
+        <alwaysOn>true</alwaysOn>
+        <updateRate>0.0</updateRate>
+        <cameraName>head_camera</cameraName>
+        <imageTopicName>rgb/image_raw</imageTopicName>
+        <cameraInfoTopicName>rgb/camera_info</cameraInfoTopicName>
+        <depthImageTopicName>depth/image_raw</depthImageTopicName>
+        <depthImageInfoTopicName>depth/camera_info</depthImageInfoTopicName>
+        <pointCloudTopicName>depth/points</pointCloudTopicName>
+        <frameName>Head_camera_link_optical</frameName>
+        <pointCloudCutoff>0.05</pointCloudCutoff>
+        <pointCloudCutoffMax>10.0</pointCloudCutoffMax>
+        <distortion_k1>0</distortion_k1>
+        <distortion_k2>0</distortion_k2>
+        <distortion_k3>0</distortion_k3>
+        <distortion_t1>0</distortion_t1>
+        <distortion_t2>0</distortion_t2>
+        <CxPrime>0</CxPrime>
+        <Cx>0</Cx>
+        <Cy>0</Cy>
+        <focalLength>0</focalLength>
+        <hackBaseline>0</hackBaseline>
+        <robotNamespace>/dual_arm</robotNamespace>
+      </plugin>
+    </sensor>
+  </gazebo>
   <link
     name="L_hip">

Commit message: feat: add yaw wrist URDF chain

File: urdf/dual_arm.urdf (robot description, URDF)
Before this commit: robot dual_arm, 27 links, 26 joints
Links:
- added link L_grip_frame
- added link L_wrist_ik_frame, mass 0.001
- added link L_wrist_yaw, mass 0.5; visual cylinder length=0.03 radius=0.017
- added link R_grip_frame
- added link R_wrist_ik_frame, mass 0.001
- added link R_wrist_yaw, mass 0.5; visual cylinder length=0.03 radius=0.017
- link L_EE: geometry collision cylinder length=0.01 radius=0.03; collision mesh filename=package://dual_arm/meshes/L_EE.STL
- link R_EE: geometry collision cylinder length=0.01 radius=0.03; collision mesh filename=package://dual_arm/meshes/R_EE.STL
Joints:
- added joint L_grip_frame_joint: type fixed, parent L_EE, child L_grip_frame, origin xyz=0.001087 -0.020925 -0.024844 rpy=0.752861 0 -2.834860
- added joint L_wrist_ik_joint: type fixed, parent L_wrist_yaw, child L_wrist_ik_frame, origin xyz=0 0 -0.10 rpy=0 0 0
- added joint L_wrist_yaw_joint: type revolute, parent L_elbow, child L_wrist_yaw, origin xyz=0 0 -0.15 rpy=0 0 0, axis 0 0 1, limit lower=-0.9 upper=0.9 effort=12 velocity=4
- added joint R_grip_frame_joint: type fixed, parent R_EE, child R_grip_frame, origin xyz=0.008658 0.029717 -0.009909 rpy=1.817146 0 2.611848
- added joint R_wrist_ik_joint: type fixed, parent R_wrist_yaw, child R_wrist_ik_frame, origin xyz=0 0 -0.10 rpy=0 0 0
- added joint R_wrist_yaw_joint: type revolute, parent R_elbow, child R_wrist_yaw, origin xyz=0 0 -0.15 rpy=0 0 0, axis 0 0 1, limit lower=-0.9 upper=0.9 effort=12 velocity=4
- joint L_EE_joint: origin xyz=0 0 -0.3 rpy=0 0 0 -> xyz=0 0 -0.15 rpy=0 0 0; parent L_elbow -> L_wrist_yaw
- joint R_EE_joint: origin xyz=0 0 -0.3 rpy=0 0 0 -> xyz=0 0 -0.15 rpy=0 0 0; parent R_elbow -> R_wrist_yaw

File: urdf/dual_arm.xacro (robot description, xacro)
@@ -341,4 +341,38 @@
       effort="30"
       velocity="8.5" />
+  </joint>
+  <!-- Mission 1: yaw-only wrist ported from jys.  The wrist link intentionally
+       has no collision geometry so it cannot strike the elbow/hand chain. -->
+  <link name="L_wrist_yaw">
+    <inertial>
+      <origin xyz="0 0 -0.015" rpy="0 0 0" />
+      <mass value="0.5" />
+      <inertia ixx="0.0025" ixy="0" ixz="0" iyy="0.0025" iyz="0" izz="0.001" />
+    </inertial>
+    <visual>
+      <origin xyz="0 0 -0.015" rpy="0 0 0" />
+      <geometry><cylinder length="0.03" radius="0.017" /></geometry>
+      <material name="wrist_dark"><color rgba="0.2 0.2 0.2 1" /></material>
+    </visual>
+  </link>
+  <joint name="L_wrist_yaw_joint" type="revolute">
+    <origin xyz="0 0 -0.15" rpy="0 0 0" />
+    <parent link="L_elbow" />
+    <child link="L_wrist_yaw" />
+    <axis xyz="0 0 1" />
+    <dynamics damping="1" />
+    <limit lower="-0.9" upper="0.9" effort="12" velocity="4" />
+  </joint>
+  <link name="L_wrist_ik_frame">
+    <inertial>
+      <origin xyz="0 0 0" rpy="0 0 0" />
+      <mass value="0.001" />
+      <inertia ixx="1E-06" ixy="0" ixz="0" iyy="1E-06" iyz="0" izz="1E-06" />
+    </inertial>
+  </link>
+  <joint name="L_wrist_ik_joint" type="fixed">
+    <origin xyz="0 0 -0.10" rpy="0 0 0" />
+    <parent link="L_wrist_yaw" />
+    <child link="L_wrist_ik_frame" />
   </joint>
   <link
@@ -434,8 +468,8 @@
     type="fixed">
     <origin
-      xyz="0 0 -0.3"
+      xyz="0 0 -0.15"
       rpy="0 0 0" />
     <parent
-      link="L_elbow" />
+      link="L_wrist_yaw" />
     <child
       link="L_EE" />
@@ -448,4 +482,11 @@
       effort="30"
       velocity="8.5" />
+  </joint>
+  <!-- Contact frame at the center and orientation of the existing jmp grip disc. -->
+  <link name="L_grip_frame" />
+  <joint name="L_grip_frame_joint" type="fixed">
+    <origin xyz="0.001087 -0.020925 -0.024844" rpy="0.752861 0 -2.834860" />
+    <parent link="L_EE" />
+    <child link="L_grip_frame" />
   </joint>
   <link
@@ -684,4 +725,37 @@
       effort="30"
       velocity="8.5" />
+  </joint>
+  <!-- Right wrist mirrors the left wrist while retaining the original jmp palm. -->
+  <link name="R_wrist_yaw">
+    <inertial>
+      <origin xyz="0 0 -0.015" rpy="0 0 0" />
+      <mass value="0.5" />
+      <inertia ixx="0.0025" ixy="0" ixz="0" iyy="0.0025" iyz="0" izz="0.001" />
+    </inertial>
+    <visual>
+      <origin xyz="0 0 -0.015" rpy="0 0 0" />
+      <geometry><cylinder length="0.03" radius="0.017" /></geometry>
+      <material name="wrist_dark"><color rgba="0.2 0.2 0.2 1" /></material>
+    </visual>
+  </link>
+  <joint name="R_wrist_yaw_joint" type="revolute">
+    <origin xyz="0 0 -0.15" rpy="0 0 0" />
+    <parent link="R_elbow" />
+    <child link="R_wrist_yaw" />
+    <axis xyz="0 0 1" />
+    <dynamics damping="1" />
+    <limit lower="-0.9" upper="0.9" effort="12" velocity="4" />
+  </joint>
+  <link name="R_wrist_ik_frame">
+    <inertial>
+      <origin xyz="0 0 0" rpy="0 0 0" />
+      <mass value="0.001" />
+      <inertia ixx="1E-06" ixy="0" ixz="0" iyy="1E-06" iyz="0" izz="1E-06" />
+    </inertial>
+  </link>
+  <joint name="R_wrist_ik_joint" type="fixed">
+    <origin xyz="0 0 -0.10" rpy="0 0 0" />
+    <parent link="R_wrist_yaw" />
+    <child link="R_wrist_ik_frame" />
   </joint>
   <link
@@ -757,8 +831,8 @@
     type="fixed">
     <origin
-      xyz="0 0 -0.3"
+      xyz="0 0 -0.15"
       rpy="0 0 0" />
     <parent
-      link="R_elbow" />
+      link="R_wrist_yaw" />
     <child
       link="R_EE" />
@@ -771,4 +845,11 @@
       effort="30"
       velocity="8.5" />
+  </joint>
+  <!-- Contact frame at the center and orientation of the existing jmp grip disc. -->
+  <link name="R_grip_frame" />
+  <joint name="R_grip_frame_joint" type="fixed">
+    <origin xyz="0.008658 0.029717 -0.009909" rpy="1.817146 0 2.611848" />
+    <parent link="R_EE" />
+    <child link="R_grip_frame" />
   </joint>
   <link
@@ -944,4 +1025,11 @@
     <provideFeedback>true</provideFeedback>
   </gazebo>
+  <!-- Use ODE's implicit damping for the new wrist axes. -->
+  <gazebo reference="L_wrist_yaw_joint">
+    <implicitSpringDamper>true</implicitSpringDamper>
+  </gazebo>
+  <gazebo reference="R_wrist_yaw_joint">
+    <implicitSpringDamper>true</implicitSpringDamper>
+  </gazebo>
   <!-- 왼쪽/오른쪽 패드 접촉 특성 변경: 기본 kp=1e12(사실상 강체)를 낮춰 접촉 시 임펄스성 반발력을
        줄이고, minDepth로 약간의 침투를 허용해 접촉 안정성을 높인다. L_EE/R_EE 링크(그립 원판이
@@ -1623,58 +1711,78 @@
   <transmission name="tran6">
     <type>transmission_interface/SimpleTransmission</type>
+    <joint name="L_wrist_yaw_joint">
+      <hardwareInterface>hardware_interface/PositionJointInterface</hardwareInterface>
+    </joint>
+    <actuator name="motor6">
+      <hardwareInterface>hardware_interface/PositionJointInterface</hardwareInterface>
+      <mechanicalReduction>50</mechanicalReduction>
+    </actuator>
+  </transmission>
+  <transmission name="tran7">
+    <type>transmission_interface/SimpleTransmission</type>
     <joint name="R_shoulder_pitch_joint">
       <hardwareInterface>hardware_interface/PositionJointInterface</hardwareInterface>
     </joint>
-    <actuator name="motor6">
+    <actuator name="motor7">
       <hardwareInterface>hardware_interface/PositionJointInterface</hardwareInterface>
       <mechanicalReduction>50</mechanicalReduction>
     </actuator>
   </transmission>
-  <transmission name="tran7">
+  <transmission name="tran8">
     <type>transmission_interface/SimpleTransmission</type>
     <joint name="R_shoulder_roll_joint">
       <hardwareInterface>hardware_interface/PositionJointInterface</hardwareInterface>
     </joint>
-    <actuator name="motor7">
+    <actuator name="motor8">
       <hardwareInterface>hardware_interface/PositionJointInterface</hardwareInterface>
       <mechanicalReduction>50</mechanicalReduction>
     </actuator>
   </transmission>
-  <transmission name="tran8">
+  <transmission name="tran9">
     <type>transmission_interface/SimpleTransmission</type>
     <joint name="R_shoulder_yaw_joint">
       <hardwareInterface>hardware_interface/PositionJointInterface</hardwareInterface>
     </joint>
-    <actuator name="motor8">
+    <actuator name="motor9">
       <hardwareInterface>hardware_interface/PositionJointInterface</hardwareInterface>
       <mechanicalReduction>50</mechanicalReduction>
     </actuator>
   </transmission>
-  <transmission name="tran9">
+  <transmission name="tran10">
     <type>transmission_interface/SimpleTransmission</type>
     <joint name="R_elbow_joint">
       <hardwareInterface>hardware_interface/PositionJointInterface</hardwareInterface>
     </joint>
-    <actuator name="motor9">
+    <actuator name="motor10">
       <hardwareInterface>hardware_interface/PositionJointInterface</hardwareInterface>
       <mechanicalReduction>50</mechanicalReduction>
     </actuator>
   </transmission>
-  <transmission name="tran10">
+  <transmission name="tran11">
+    <type>transmission_interface/SimpleTransmission</type>
+    <joint name="R_wrist_yaw_joint">
+      <hardwareInterface>hardware_interface/PositionJointInterface</hardwareInterface>
+    </joint>
+    <actuator name="motor11">
+      <hardwareInterface>hardware_interface/PositionJointInterface</hardwareInterface>
+      <mechanicalReduction>50</mechanicalReduction>
+    </actuator>
+  </transmission>
+  <transmission name="tran12">
     <type>transmission_interface/SimpleTransmission</type>
     <joint name="Head_yaw_joint">
       <hardwareInterface>hardware_interface/PositionJointInterface</hardwareInterface>
     </joint>
-    <actuator name="motor10">
+    <actuator name="motor12">
       <hardwareInterface>hardware_interface/PositionJointInterface</hardwareInterface>
       <mechanicalReduction>50</mechanicalReduction>
     </actuator>
   </transmission>
-  <transmission name="tran11">
+  <transmission name="tran13">
     <type>transmission_interface/SimpleTransmission</type>
     <joint name="Head_pitch_joint">
       <hardwareInterface>hardware_interface/PositionJointInterface</hardwareInterface>
     </joint>
-    <actuator name="motor11">
+    <actuator name="motor13">
       <hardwareInterface>hardware_interface/PositionJointInterface</hardwareInterface>
       <mechanicalReduction>50</mechanicalReduction>
@@ -1734,58 +1842,78 @@
   <transmission name="tran6">
     <type>transmission_interface/SimpleTransmission</type>
+    <joint name="L_wrist_yaw_joint">
+      <hardwareInterface>hardware_interface/EffortJointInterface</hardwareInterface>
+    </joint>
+    <actuator name="motor6">
+      <hardwareInterface>hardware_interface/EffortJointInterface</hardwareInterface>
+      <mechanicalReduction>1</mechanicalReduction>
+    </actuator>
+  </transmission>
+  <transmission name="tran7">
+    <type>transmission_interface/SimpleTransmission</type>
     <joint name="R_shoulder_pitch_joint">
       <hardwareInterface>hardware_interface/EffortJointInterface</hardwareInterface>
     </joint>
-    <actuator name="motor6">
+    <actuator name="motor7">
       <hardwareInterface>hardware_interface/EffortJointInterface</hardwareInterface>
       <mechanicalReduction>1</mechanicalReduction>
     </actuator>
   </transmission>
-  <transmission name="tran7">
+  <transmission name="tran8">
     <type>transmission_interface/SimpleTransmission</type>
     <joint name="R_shoulder_roll_joint">
       <hardwareInterface>hardware_interface/EffortJointInterface</hardwareInterface>
     </joint>
-    <actuator name="motor7">
+    <actuator name="motor8">
       <hardwareInterface>hardware_interface/EffortJointInterface</hardwareInterface>
       <mechanicalReduction>1</mechanicalReduction>
     </actuator>
   </transmission>
-  <transmission name="tran8">
+  <transmission name="tran9">
     <type>transmission_interface/SimpleTransmission</type>
     <joint name="R_shoulder_yaw_joint">
       <hardwareInterface>hardware_interface/EffortJointInterface</hardwareInterface>
     </joint>
-    <actuator name="motor8">
+    <actuator name="motor9">
       <hardwareInterface>hardware_interface/EffortJointInterface</hardwareInterface>
       <mechanicalReduction>1</mechanicalReduction>
     </actuator>
   </transmission>
-  <transmission name="tran9">
+  <transmission name="tran10">
     <type>transmission_interface/SimpleTransmission</type>
     <joint name="R_elbow_joint">
       <hardwareInterface>hardware_interface/EffortJointInterface</hardwareInterface>
     </joint>
-    <actuator name="motor9">
+    <actuator name="motor10">
       <hardwareInterface>hardware_interface/EffortJointInterface</hardwareInterface>
       <mechanicalReduction>1</mechanicalReduction>
     </actuator>
   </transmission>
-  <transmission name="tran10">
+  <transmission name="tran11">
+    <type>transmission_interface/SimpleTransmission</type>
+    <joint name="R_wrist_yaw_joint">
+      <hardwareInterface>hardware_interface/EffortJointInterface</hardwareInterface>
+    </joint>
+    <actuator name="motor11">
+      <hardwareInterface>hardware_interface/EffortJointInterface</hardwareInterface>
+      <mechanicalReduction>1</mechanicalReduction>
+    </actuator>
+  </transmission>
+  <transmission name="tran12">
     <type>transmission_interface/SimpleTransmission</type>
     <joint name="Head_yaw_joint">
       <hardwareInterface>hardware_interface/EffortJointInterface</hardwareInterface>
     </joint>
-    <actuator name="motor10">
+    <actuator name="motor12">
       <hardwareInterface>hardware_interface/EffortJointInterface</hardwareInterface>
       <mechanicalReduction>1</mechanicalReduction>
     </actuator>
   </transmission>
-  <transmission name="tran11">
+  <transmission name="tran13">
     <type>transmission_interface/SimpleTransmission</type>
     <joint name="Head_pitch_joint">
       <hardwareInterface>hardware_interface/EffortJointInterface</hardwareInterface>
     </joint>
-    <actuator name="motor11">
+    <actuator name="motor13">
       <hardwareInterface>hardware_interface/EffortJointInterface</hardwareInterface>
       <mechanicalReduction>1</mechanicalReduction>
