Commit message: feat: L/R 손목 yaw 관절 추가, 그립 패드를 원판에서 평면 박스로 교체
배경/문제:
고정 원판 패드는 오프라인 스크립트로 계산한 rpy가 "그 순간 그 자세 하나"에만
맞는 상수값이라, waist 각도나 접근 자세가 달라지면 다시 어긋난다. 손목 관절
없이는 손 방향이 IK task에 아예 안 들어가 있어 근본적으로 고칠 수 없는
구조였음. 이 문제를 풀기 위한 5단계 계획(wrist-compliance-port)의 1번
과제로, 아직 컨트롤러/트랜스미션은 없는 순수 URDF/기구 레이어 변경.

검토한 대안과 선택 이유:
별도 브랜치 jys에 이미 작동하는 손목 컴플라이언스 구현이 있으나(merge-base가
초기 커밋 수준이라 diff/cherry-pick 불가) 개념만 이식해 이 브랜치의 기존
구조(멀티라인 속성 스타일의 원본 SolidWorks-export 블록과, 최근 그립 패드
핫픽스 커밋들이 쓴 컴팩트 한 줄 스타일이 혼재) 위에 재구현. 손목 체인/팜
콜리전 삽입은 계획서(브리핑)가 제시한 XML을 그대로 채택했고, 그 안의
"-- this is a placeholder..." 주석 문구에 있던 이중 하이픈만 XML 주석
규칙 위반(expat: not well-formed)이라 단일 하이픈으로 수정했다.

구현 내용:
urdf/dual_arm.xacro의 L_elbow/R_elbow -> L_EE/R_EE 직결을 L_elbow ->
L_wrist_yaw_joint(revolute, axis z, ±0.9rad, damping 1) -> L_wrist_yaw ->
{L_wrist_ik_joint(고정, IK 전용) -> L_wrist_ik_frame, L_EE_joint(고정,
기존 grasp_offset 수학이 model.getFrameId("L_EE_joint")로 타겟하는 nominal
프레임 이름/시맨틱 그대로 유지) -> L_EE} 구조로 변경. L_EE의 충돌 형상을
기존 STL mesh 콜리전 + 원판 그립패드 콜리전 조합에서 평면 박스 하나
(0.090x0.025x0.090, origin 0 -0.0375 -0.005)로 교체하고, 그 자리를 그대로
쓰는 L_grip_frame(빈 링크, L_grip_joint로 L_EE의 자식)을 접촉/admittance
기준 프레임으로 추가. R arm도 Y부호만 뒤집어(+0.0375) 동일 대칭 구조로
미러링 - 기존 L/R 미러링 컨벤션(예: L_elbow/R_elbow inertial y부호)과 일치.
더 이상 존재하지 않는 원판 패드의 rpy 보정 이력을 설명하던 옛 한국어 주석
(fk_debug.cpp/fk_pad_calc.cpp/recompute_pad_rpy.py/compute_tangent_offset.py
관련)은 이번 변경으로 삭제되는 코드를 그대로 설명하던 것이라 함께 제거.
mu1/mu2/kp/kd/minDepth 게조보 접촉 튜닝과 lumping-disable/FT센서 블록은
링크명(L_EE/R_EE)/조인트명(L_EE_joint/R_EE_joint) 기준으로 이미 걸려있어
수정 없이 그대로 적용됨을 grep으로 확인. tran1~tran10 트랜스미션 블록은
L_elbow_joint/R_elbow_joint까지만 다뤄 새 wrist 조인트엔 아직 액추에이터가
없음(Task 2 몫)도 확인.

결과/검증:
xacro urdf/dual_arm.xacro > urdf/dual_arm.urdf로 재생성 (에러 없음, 출력도
XML 재파싱 성공). pinocchio buildModelFromUrdf로 로드해 nq=nv=13 확인.
model.names 실측 순서는 (pinocchio 관례상 index 0이 항상 "universe")
1:Waist_joint 2:Head_yaw_joint 3:Head_pitch_joint 4:L_shoulder_pitch_joint
5:L_shoulder_roll_joint 6:L_shoulder_yaw_joint 7:L_elbow_joint
8:L_wrist_yaw_joint 9:R_shoulder_pitch_joint 10:R_shoulder_roll_joint
11:R_shoulder_yaw_joint 12:R_elbow_joint 13:R_wrist_yaw_joint - universe
오프셋(+1)을 감안하면 태스크 계획서가 예측한 순서(0:Waist...12:R_wy)와
정확히 일치. L_wrist_ik_joint/R_wrist_ik_joint/L_EE_joint/R_EE_joint/
L_grip_joint/R_grip_joint 전부 getFrameId 결과가 model.nframes(66)보다
작은 유효 인덱스(44/46/48/60/62/64)임을 확인. Gazebo 실행 검증은 다음
태스크(컨트롤러/트랜스미션 추가) 이후로 미룸 - 지금 상태로는 새 관절에
액추에이터가 없어 아직 못 띄움.

File: urdf/dual_arm.urdf (robot description, URDF)
Before this commit: robot dual_arm, 27 links, 26 joints
Links:
- added link L_grip_frame
- added link L_wrist_ik_frame, mass 0.001
- added link L_wrist_yaw, mass 0.5; visual cylinder length=0.03 radius=0.017
- added link R_grip_frame
- added link R_wrist_ik_frame, mass 0.001
- added link R_wrist_yaw, mass 0.5; visual cylinder length=0.03 radius=0.017
- link L_EE: geometry collision box size=0.090 0.025 0.090; visual box size=0.090 0.025 0.090
- link R_EE: geometry collision box size=0.090 0.025 0.090; visual box size=0.090 0.025 0.090
Joints:
- added joint L_grip_joint: type fixed, parent L_EE, child L_grip_frame, origin xyz=0 -0.0375 -0.005 rpy=0 0 0
- added joint L_wrist_ik_joint: type fixed, parent L_wrist_yaw, child L_wrist_ik_frame, origin xyz=0 0 -0.10 rpy=0 0 0
- added joint L_wrist_yaw_joint: type revolute, parent L_elbow, child L_wrist_yaw, origin xyz=0 0 -0.15 rpy=0 0 0, axis 0 0 1, limit lower=-0.9 upper=0.9 effort=12 velocity=4.0
- added joint R_grip_joint: type fixed, parent R_EE, child R_grip_frame, origin xyz=0 0.0375 -0.005 rpy=0 0 0
- added joint R_wrist_ik_joint: type fixed, parent R_wrist_yaw, child R_wrist_ik_frame, origin xyz=0 0 -0.10 rpy=0 0 0
- added joint R_wrist_yaw_joint: type revolute, parent R_elbow, child R_wrist_yaw, origin xyz=0 0 -0.15 rpy=0 0 0, axis 0 0 1, limit lower=-0.9 upper=0.9 effort=12 velocity=4.0
- joint L_EE_joint: axis 0 0 0 -> (none); limit lower=-1.57 upper=1.57 effort=30 velocity=8.5 -> (none); origin xyz=0 0 -0.3 rpy=0 0 0 -> xyz=0 0 -0.15 rpy=0 0 0; parent L_elbow -> L_wrist_yaw
- joint R_EE_joint: axis 0 0 0 -> (none); limit lower=-1.57 upper=1.57 effort=30 velocity=8.5 -> (none); origin xyz=0 0 -0.3 rpy=0 0 0 -> xyz=0 0 -0.15 rpy=0 0 0; parent R_elbow -> R_wrist_yaw

File: urdf/dual_arm.xacro (robot description, xacro)
@@ -342,110 +342,77 @@
       velocity="8.5" />
   </joint>
-  <link
-    name="L_EE">
-    <inertial>
-      <origin
-        xyz="0 0 -0.003514"
-        rpy="0 0 0" />
-      <mass
-        value="0.15" />
-      <inertia
-        ixx="5.5E-05"
-        ixy="0"
-        ixz="0"
-        iyy="5.5E-05"
-        iyz="0"
-        izz="6.4E-05" />
-    </inertial>
-    <visual>
-      <origin
-        xyz="0 0 0"
-        rpy="0 0 0" />
-      <geometry>
-        <mesh
-          filename="package://dual_arm/meshes/L_EE.STL" />
-      </geometry>
-      <material
-        name="">
-        <color
-          rgba="0.298039215686275 0.298039215686275 0.298039215686275 1" />
-      </material>
-    </visual>
-    <collision>
-      <origin
-        xyz="0 0 0"
-        rpy="0 0 0" />
-      <geometry>
-        <mesh
-          filename="package://dual_arm/meshes/L_EE.STL" />
-      </geometry>
-    </collision>
-    <!-- 파지 안정성 보강용 평면 접촉 패드. L_EE.STL은 실측(메시 직접 파싱) 결과 약 6.5x6.5x5.4cm의
-         거의 구형(반경 ~3.25cm)이라 박스 평면과 사실상 점 접촉만 생겨 이송 중 자세가 흔들리기 쉽다.
-         2026-07-13 admittance 검증(F/T 로그) 중 좌/우 힘이 크게 비대칭(예: 같은 tick에 R이 -27N인데
-         L은 +7.5N)으로 나타나 물체가 회전하며 낙하하는 게 확인됐고, fk_debug(실제 SolveIK_Position/
-         grasp_offset=0.040/STANDOFF_Y=0.15 그대로 재현)로 다시 재보니 L_EE 로컬 Y축이 스퀴즈
-         방향(월드 Y축)과 dot=0.757(약 40.8° 어긋남) - 이전 주석의 dot~0.77(grasp_offset=0.043 기준)
-         수치는 grasp_offset이 0.040으로 바뀌면서 이미 stale이었다. 패드가 로컬 Y로 고정돼 있어
-         면 접촉이 아니라 모서리 접촉에 가까웠던 것으로 보고, rpy를 EE 로컬 프레임에서 "월드 Y가
-         가리키는 실제 방향"(target_local_dir = R_EE^T * worldY)으로 패드 법선이 향하도록 보정한다
-         (계산: fk_debug.cpp, 일회성 도구, 커밋 안 함). 위치(xyz)는 그대로 두고 방향만 보정 -
-         정확한 돌출거리 재튜닝(전체 손 형상 재설계, P2)은 이후 과제로 보류. -->
-    <!-- 원형 접촉 패드: 기존 사각 패드(box)+L자형 턱 조합을 하나의 평평한 원판(cylinder)으로 교체.
-         rpy는 실제 vision pick 파이프라인(base_seed=0 스폰 상태 -> segment 1 standoff -> segment 1b
-         접촉, main.cpp와 동일한 SolveIK_Position/CartesianLineTrajectory/grasp_offset=0.040/
-         STANDOFF_Y=0.15/v_des를 그대로 재현)을 처음부터 다시 풀어서, 실제 파지 순간 L_EE 프레임의
-         world 자세를 구한 뒤, 원판 법선(로컬 Z축)이 파지 시점 물체 옆면 법선(월드 Y축)과 정확히
-         평행해지는 방향으로 역산했다 (계산: fk_pad_calc.cpp, 일회성 도구, 커밋 안 함, dot=1.0 검증).
-         위치(origin xyz)는 기존 패드 자리를 그대로 재사용 - mesh 표면 돌출거리 재튜닝은 보류.
-         2026-07-17(1): SolveIK_Position에 null-space q_pref(elbow-down+out) 투영을 추가하면서
-         파지 시점 실제 손 자세가 달라져 rpy를 재계산했다(recompute_pad_rpy.py, 일회성 도구,
-         커밋 안 함, dot=1.0 재검증) - null-space 항이 관절 배치를 바꾸면 이 rpy도 다시 맞춰야 한다.
-         2026-07-17(2): origin xyz를 "탄젠트 접점" 방식으로 재계산했다(compute_tangent_offset.py,
-         일회성 도구, 커밋 안 함) - 기존엔 이전 사각패드 자리를 관성적으로 재사용/스케일링만 해왔는데,
-         Gazebo에서 패드가 손목 mesh에 파묻히거나 반대로 붕 뜨는 문제가 반복됐다. L_EE/R_EE 원점
-         (손목 구체 중심)에서 물체 중심 방향으로, 월드 Z성분을 0으로 강제한(손목 구체 중앙 높이
-         유지) 뒤 손목 구체 실측 반지름(0.0325m)만큼 나간 지점을 월드 좌표로 구하고, 이를 손
-         로컬 프레임으로 역변환해 origin xyz로 썼다 - 원판이 손목 구체 표면에 기하학적으로 정확히
-         접하도록(붕 뜸도 파묻힘도 없이) 만드는 게 목적. rpy는 그 후 사용자가 Gazebo 육안 확인으로
-         왼쪽 +7.5°/오른쪽 -7.5°(대칭) 미세 조정해 최종 확정했다. -->
-    <visual name="L_EE_grip_disc_visual">
-      <origin
-        xyz="0.001087 -0.020925 -0.024844"
-        rpy="0.752861 -0.000000 -2.834860" />
-      <geometry>
-        <cylinder radius="0.03" length="0.01" />
-      </geometry>
-      <material name="grip_pad_orange">
-        <color rgba="1.0 0.5 0.0 1" />
-      </material>
-    </visual>
-    <collision name="L_EE_grip_disc_collision">
-      <origin
-        xyz="0.001087 -0.020925 -0.024844"
-        rpy="0.752861 -0.000000 -2.834860" />
-      <geometry>
-        <cylinder radius="0.03" length="0.01" />
-      </geometry>
-    </collision>
-  </link>
-  <joint
-    name="L_EE_joint"
-    type="fixed">
-    <origin
-      xyz="0 0 -0.3"
-      rpy="0 0 0" />
-    <parent
-      link="L_elbow" />
-    <child
-      link="L_EE" />
-    <axis
-      xyz="0 0 0" />
-    <dynamics damping="1"/>
-    <limit
-      lower="-1.57"
-      upper="1.57"
-      effort="30"
-      velocity="8.5" />
+  <link name="L_wrist_yaw">
+    <inertial>
+      <origin xyz="0 0 -0.015" rpy="0 0 0" />
+      <mass value="0.5" />
+      <inertia ixx="2.5E-03" ixy="0" ixz="0" iyy="2.5E-03" iyz="0" izz="1.0E-03" />
+    </inertial>
+    <visual>
+      <origin xyz="0 0 -0.015" rpy="0 0 0" />
+      <geometry><cylinder radius="0.017" length="0.03" /></geometry>
+      <material name="wrist_dark"><color rgba="0.18 0.18 0.18 1" /></material>
+    </visual>
+    <!-- No collision on this link: STL mesh + wrist + pad collisions overlapping
+         caused Gazebo startup instability in jys's testing. Keep collision only
+         on L_EE below. -->
+  </link>
+  <joint name="L_wrist_yaw_joint" type="revolute">
+    <origin xyz="0 0 -0.15" rpy="0 0 0" />
+    <parent link="L_elbow" />
+    <child link="L_wrist_yaw" />
+    <axis xyz="0 0 1" />
+    <dynamics damping="1" />
+    <limit lower="-0.9" upper="0.9" effort="12" velocity="4.0" />
+  </joint>
+  <!-- Fixed IK-only frame: give it a tiny nonzero inertial or ODE's fixed-joint
+       lumping can become ill-conditioned with a controlled joint upstream. -->
+  <link name="L_wrist_ik_frame">
+    <inertial>
+      <origin xyz="0 0 0" rpy="0 0 0" />
+      <mass value="0.001" />
+      <inertia ixx="1.0E-06" ixy="0" ixz="0" iyy="1.0E-06" iyz="0" izz="1.0E-06" />
+    </inertial>
+  </link>
+  <joint name="L_wrist_ik_joint" type="fixed">
+    <origin xyz="0 0 -0.10" rpy="0 0 0" />
+    <parent link="L_wrist_yaw" />
+    <child link="L_wrist_ik_frame" />
+  </joint>
+  <link name="L_EE">
+    <inertial>
+      <origin xyz="0 0 -0.003514" rpy="0 0 0" />
+      <mass value="0.15" />
+      <inertia ixx="5.5E-05" ixy="0" ixz="0" iyy="5.5E-05" iyz="0" izz="6.4E-05" />
+    </inertial>
+    <visual>
+      <origin xyz="0 0 0" rpy="0 0 0" />
+      <geometry><mesh filename="package://dual_arm/meshes/L_EE.STL" /></geometry>
+      <material name=""><color rgba="0.298039215686275 0.298039215686275 0.298039215686275 1" /></material>
+    </visual>
+    <!-- Single flat palm collision replaces the old STL-mesh + disc-pad combo.
+         Offset/size copied from jys (0.090 x 0.025 x 0.090 box, 3.75cm out in -Y,
+         0.5cm down) - this is a placeholder mount pose to be re-tuned in Task 6
+         against this branch's actual arm geometry, same way the old disc pad
+         needed 3 rounds of offline recomputation. -->
+    <collision name="L_EE_palm_collision">
+      <origin xyz="0 -0.0375 -0.005" rpy="0 0 0" />
+      <geometry><box size="0.090 0.025 0.090" /></geometry>
+    </collision>
+    <visual name="L_EE_grip_pad_visual">
+      <origin xyz="0 -0.0375 -0.005" rpy="0 0 0" />
+      <geometry><box size="0.090 0.025 0.090" /></geometry>
+      <material name="grip_pad_visual_dark"><color rgba="0.12 0.12 0.12 1" /></material>
+    </visual>
+  </link>
+  <joint name="L_EE_joint" type="fixed">
+    <origin xyz="0 0 -0.15" rpy="0 0 0" />
+    <parent link="L_wrist_yaw" />
+    <child link="L_EE" />
+  </joint>
+  <link name="L_grip_frame" />
+  <joint name="L_grip_joint" type="fixed">
+    <origin xyz="0 -0.0375 -0.005" rpy="0 0 0" />
+    <parent link="L_EE" />
+    <child link="L_grip_frame" />
   </joint>
   <link
@@ -685,90 +652,77 @@
       velocity="8.5" />
   </joint>
-  <link
-    name="R_EE">
-    <inertial>
-      <origin
-        xyz="0 0 -0.003514"
-        rpy="0 0 0" />
-      <mass
-        value="0.15" />
-      <inertia
-        ixx="5.5E-05"
-        ixy="0"
-        ixz="0"
-        iyy="5.5E-05"
-        iyz="0"
-        izz="6.4E-05" />
-    </inertial>
-    <visual>
-      <origin
-        xyz="0 0 0"
-        rpy="0 0 0" />
-      <geometry>
-        <mesh
-          filename="package://dual_arm/meshes/R_EE.STL" />
-      </geometry>
-      <material
-        name="">
-        <color
-          rgba="0.298039215686275 0.298039215686275 0.298039215686275 1" />
-      </material>
-    </visual>
-    <collision>
-      <origin
-        xyz="0 0 0"
-        rpy="0 0 0" />
-      <geometry>
-        <mesh
-          filename="package://dual_arm/meshes/R_EE.STL" />
-      </geometry>
-    </collision>
-    <!-- 파지 안정성 보강용 평면 접촉 패드 (L_EE 쪽 설명 참고, mesh 반경 ~3.25cm). 이전 주석은
-         "R_EE 로컬 Y축이 dot~0.99로 거의 완벽히 정렬"이라고 기록했으나, 이는 grasp_offset=0.043
-         기준 stale 수치였다. 2026-07-13 fk_debug(현재 코드의 grasp_offset=0.040/STANDOFF_Y=0.15
-         그대로 재현)로 재계산하니 실제로는 dot=0.955(약 17.2° 어긋남) - L_EE(40.8°)보다는 낫지만
-         무시할 수준은 아니다. L_EE와 동일한 방식으로 rpy를 target_local_dir(=R_EE^T*worldY)에
-         맞춰 보정한다 (계산: fk_debug.cpp, 일회성 도구, 커밋 안 함). -->
-    <!-- 원형 접촉 패드 - L_EE 쪽 설명 참고. 동일한 방식(recompute_pad_rpy.py로 null-space
-         적용된 파지 파이프라인 처음부터 재현, compute_tangent_offset.py로 탄젠트 접점 위치
-         재계산)으로 rpy/xyz 재계산, dot=1.0 검증. rpy 최종값은 왼쪽과 대칭으로 -7.5° 미세 조정. -->
-    <visual name="R_EE_grip_disc_visual">
-      <origin
-        xyz="0.008658 0.029717 -0.009909"
-        rpy="1.817146 -0.000000 2.611848" />
-      <geometry>
-        <cylinder radius="0.03" length="0.01" />
-      </geometry>
-      <material name="grip_pad_orange">
-        <color rgba="1.0 0.5 0.0 1" />
-      </material>
-    </visual>
-    <collision name="R_EE_grip_disc_collision">
-      <origin
-        xyz="0.008658 0.029717 -0.009909"
-        rpy="1.817146 -0.000000 2.611848" />
-      <geometry>
-        <cylinder radius="0.03" length="0.01" />
-      </geometry>
-    </collision>
-  </link>
-  <joint
-    name="R_EE_joint"
-    type="fixed">
-    <origin
-      xyz="0 0 -0.3"
-      rpy="0 0 0" />
-    <parent
-      link="R_elbow" />
-    <child
-      link="R_EE" />
-    <axis
-      xyz="0 0 0" />
-    <dynamics damping="1"/>
-    <limit
-      lower="-1.57"
-      upper="1.57"
-      effort="30"
-      velocity="8.5" />
+  <link name="R_wrist_yaw">
+    <inertial>
+      <origin xyz="0 0 -0.015" rpy="0 0 0" />
+      <mass value="0.5" />
+      <inertia ixx="2.5E-03" ixy="0" ixz="0" iyy="2.5E-03" iyz="0" izz="1.0E-03" />
+    </inertial>
+    <visual>
+      <origin xyz="0 0 -0.015" rpy="0 0 0" />
+      <geometry><cylinder radius="0.017" length="0.03" /></geometry>
+      <material name="wrist_dark"><color rgba="0.18 0.18 0.18 1" /></material>
+    </visual>
+    <!-- No collision on this link: STL mesh + wrist + pad collisions overlapping
+         caused Gazebo startup instability in jys's testing. Keep collision only
+         on R_EE below. -->
+  </link>
+  <joint name="R_wrist_yaw_joint" type="revolute">
+    <origin xyz="0 0 -0.15" rpy="0 0 0" />
+    <parent link="R_elbow" />
+    <child link="R_wrist_yaw" />
+    <axis xyz="0 0 1" />
+    <dynamics damping="1" />
+    <limit lower="-0.9" upper="0.9" effort="12" velocity="4.0" />
+  </joint>
+  <!-- Fixed IK-only frame: give it a tiny nonzero inertial or ODE's fixed-joint
+       lumping can become ill-conditioned with a controlled joint upstream. -->
+  <link name="R_wrist_ik_frame">
+    <inertial>
+      <origin xyz="0 0 0" rpy="0 0 0" />
+      <mass value="0.001" />
+      <inertia ixx="1.0E-06" ixy="0" ixz="0" iyy="1.0E-06" iyz="0" izz="1.0E-06" />
+    </inertial>
+  </link>
+  <joint name="R_wrist_ik_joint" type="fixed">
+    <origin xyz="0 0 -0.10" rpy="0 0 0" />
+    <parent link="R_wrist_yaw" />
+    <child link="R_wrist_ik_frame" />
+  </joint>
+  <link name="R_EE">
+    <inertial>
+      <origin xyz="0 0 -0.003514" rpy="0 0 0" />
+      <mass value="0.15" />
+      <inertia ixx="5.5E-05" ixy="0" ixz="0" iyy="5.5E-05" iyz="0" izz="6.4E-05" />
+    </inertial>
+    <visual>
+      <origin xyz="0 0 0" rpy="0 0 0" />
+      <geometry><mesh filename="package://dual_arm/meshes/R_EE.STL" /></geometry>
+      <material name=""><color rgba="0.298039215686275 0.298039215686275 0.298039215686275 1" /></material>
+    </visual>
+    <!-- Single flat palm collision replaces the old STL-mesh + disc-pad combo.
+         Offset/size copied from jys (0.090 x 0.025 x 0.090 box, 3.75cm out in +Y,
+         0.5cm down) - this is a placeholder mount pose to be re-tuned in Task 6
+         against this branch's actual arm geometry, same way the old disc pad
+         needed 3 rounds of offline recomputation. -->
+    <collision name="R_EE_palm_collision">
+      <origin xyz="0 0.0375 -0.005" rpy="0 0 0" />
+      <geometry><box size="0.090 0.025 0.090" /></geometry>
+    </collision>
+    <visual name="R_EE_grip_pad_visual">
+      <origin xyz="0 0.0375 -0.005" rpy="0 0 0" />
+      <geometry><box size="0.090 0.025 0.090" /></geometry>
+      <material name="grip_pad_visual_dark"><color rgba="0.12 0.12 0.12 1" /></material>
+    </visual>
+  </link>
+  <joint name="R_EE_joint" type="fixed">
+    <origin xyz="0 0 -0.15" rpy="0 0 0" />
+    <parent link="R_wrist_yaw" />
+    <child link="R_EE" />
+  </joint>
+  <link name="R_grip_frame" />
+  <joint name="R_grip_joint" type="fixed">
+    <origin xyz="0 0.0375 -0.005" rpy="0 0 0" />
+    <parent link="R_EE" />
+    <child link="R_grip_frame" />
   </joint>
   <link

Commit message: feat: generalize mirrored palm contact pads

File: urdf/dual_arm.urdf (robot description, URDF)
Before this commit: robot dual_arm, 33 links, 32 joints
Joints:
- joint L_grip_frame_joint: origin xyz=0.001087 -0.020925 -0.024844 rpy=0.752861 0 -2.834860 -> xyz=0 -0.0325 0 rpy=1.57079632679 0 0
- joint R_grip_frame_joint: origin xyz=0.008658 0.029717 -0.009909 rpy=1.817146 0 2.611848 -> xyz=0 0.0325 0 rpy=-1.57079632679 0 0

File: urdf/dual_arm.xacro (robot description, xacro)
@@ -415,37 +415,11 @@
       </geometry>
     </collision>
-    <!-- 파지 안정성 보강용 평면 접촉 패드. L_EE.STL은 실측(메시 직접 파싱) 결과 약 6.5x6.5x5.4cm의
-         거의 구형(반경 ~3.25cm)이라 박스 평면과 사실상 점 접촉만 생겨 이송 중 자세가 흔들리기 쉽다.
-         2026-07-13 admittance 검증(F/T 로그) 중 좌/우 힘이 크게 비대칭(예: 같은 tick에 R이 -27N인데
-         L은 +7.5N)으로 나타나 물체가 회전하며 낙하하는 게 확인됐고, fk_debug(실제 SolveIK_Position/
-         grasp_offset=0.040/STANDOFF_Y=0.15 그대로 재현)로 다시 재보니 L_EE 로컬 Y축이 스퀴즈
-         방향(월드 Y축)과 dot=0.757(약 40.8° 어긋남) - 이전 주석의 dot~0.77(grasp_offset=0.043 기준)
-         수치는 grasp_offset이 0.040으로 바뀌면서 이미 stale이었다. 패드가 로컬 Y로 고정돼 있어
-         면 접촉이 아니라 모서리 접촉에 가까웠던 것으로 보고, rpy를 EE 로컬 프레임에서 "월드 Y가
-         가리키는 실제 방향"(target_local_dir = R_EE^T * worldY)으로 패드 법선이 향하도록 보정한다
-         (계산: fk_debug.cpp, 일회성 도구, 커밋 안 함). 위치(xyz)는 그대로 두고 방향만 보정 -
-         정확한 돌출거리 재튜닝(전체 손 형상 재설계, P2)은 이후 과제로 보류. -->
-    <!-- 원형 접촉 패드: 기존 사각 패드(box)+L자형 턱 조합을 하나의 평평한 원판(cylinder)으로 교체.
-         rpy는 실제 vision pick 파이프라인(base_seed=0 스폰 상태 -> segment 1 standoff -> segment 1b
-         접촉, main.cpp와 동일한 SolveIK_Position/CartesianLineTrajectory/grasp_offset=0.040/
-         STANDOFF_Y=0.15/v_des를 그대로 재현)을 처음부터 다시 풀어서, 실제 파지 순간 L_EE 프레임의
-         world 자세를 구한 뒤, 원판 법선(로컬 Z축)이 파지 시점 물체 옆면 법선(월드 Y축)과 정확히
-         평행해지는 방향으로 역산했다 (계산: fk_pad_calc.cpp, 일회성 도구, 커밋 안 함, dot=1.0 검증).
-         위치(origin xyz)는 기존 패드 자리를 그대로 재사용 - mesh 표면 돌출거리 재튜닝은 보류.
-         2026-07-17(1): SolveIK_Position에 null-space q_pref(elbow-down+out) 투영을 추가하면서
-         파지 시점 실제 손 자세가 달라져 rpy를 재계산했다(recompute_pad_rpy.py, 일회성 도구,
-         커밋 안 함, dot=1.0 재검증) - null-space 항이 관절 배치를 바꾸면 이 rpy도 다시 맞춰야 한다.
-         2026-07-17(2): origin xyz를 "탄젠트 접점" 방식으로 재계산했다(compute_tangent_offset.py,
-         일회성 도구, 커밋 안 함) - 기존엔 이전 사각패드 자리를 관성적으로 재사용/스케일링만 해왔는데,
-         Gazebo에서 패드가 손목 mesh에 파묻히거나 반대로 붕 뜨는 문제가 반복됐다. L_EE/R_EE 원점
-         (손목 구체 중심)에서 물체 중심 방향으로, 월드 Z성분을 0으로 강제한(손목 구체 중앙 높이
-         유지) 뒤 손목 구체 실측 반지름(0.0325m)만큼 나간 지점을 월드 좌표로 구하고, 이를 손
-         로컬 프레임으로 역변환해 origin xyz로 썼다 - 원판이 손목 구체 표면에 기하학적으로 정확히
-         접하도록(붕 뜸도 파묻힘도 없이) 만드는 게 목적. rpy는 그 후 사용자가 Gazebo 육안 확인으로
-         왼쪽 +7.5°/오른쪽 -7.5°(대칭) 미세 조정해 최종 확정했다. -->
+    <!-- Pose-independent grip pad: its normal is exactly the EE local -Y axis.
+         The mirrored right pad uses +Y.  No world-frame IK pose is baked into
+         this geometry, so wrist compliance can align it to the object surface. -->
     <visual name="L_EE_grip_disc_visual">
       <origin
-        xyz="0.001087 -0.020925 -0.024844"
-        rpy="0.752861 -0.000000 -2.834860" />
+        xyz="0 -0.0325 0"
+        rpy="1.57079632679 0 0" />
       <geometry>
         <cylinder radius="0.03" length="0.01" />
@@ -457,6 +431,6 @@
     <collision name="L_EE_grip_disc_collision">
       <origin
-        xyz="0.001087 -0.020925 -0.024844"
-        rpy="0.752861 -0.000000 -2.834860" />
+        xyz="0 -0.0325 0"
+        rpy="1.57079632679 0 0" />
       <geometry>
         <cylinder radius="0.03" length="0.01" />
@@ -483,8 +457,8 @@
       velocity="8.5" />
   </joint>
-  <!-- Contact frame at the center and orientation of the existing jmp grip disc. -->
+  <!-- Contact frame at the center and orientation of the neutral grip disc. -->
   <link name="L_grip_frame" />
   <joint name="L_grip_frame_joint" type="fixed">
-    <origin xyz="0.001087 -0.020925 -0.024844" rpy="0.752861 0 -2.834860" />
+    <origin xyz="0 -0.0325 0" rpy="1.57079632679 0 0" />
     <parent link="L_EE" />
     <child link="L_grip_frame" />
@@ -798,17 +772,9 @@
       </geometry>
     </collision>
-    <!-- 파지 안정성 보강용 평면 접촉 패드 (L_EE 쪽 설명 참고, mesh 반경 ~3.25cm). 이전 주석은
-         "R_EE 로컬 Y축이 dot~0.99로 거의 완벽히 정렬"이라고 기록했으나, 이는 grasp_offset=0.043
-         기준 stale 수치였다. 2026-07-13 fk_debug(현재 코드의 grasp_offset=0.040/STANDOFF_Y=0.15
-         그대로 재현)로 재계산하니 실제로는 dot=0.955(약 17.2° 어긋남) - L_EE(40.8°)보다는 낫지만
-         무시할 수준은 아니다. L_EE와 동일한 방식으로 rpy를 target_local_dir(=R_EE^T*worldY)에
-         맞춰 보정한다 (계산: fk_debug.cpp, 일회성 도구, 커밋 안 함). -->
-    <!-- 원형 접촉 패드 - L_EE 쪽 설명 참고. 동일한 방식(recompute_pad_rpy.py로 null-space
-         적용된 파지 파이프라인 처음부터 재현, compute_tangent_offset.py로 탄젠트 접점 위치
-         재계산)으로 rpy/xyz 재계산, dot=1.0 검증. rpy 최종값은 왼쪽과 대칭으로 -7.5° 미세 조정. -->
+    <!-- Pose-independent mirrored grip pad; normal is the EE local +Y axis. -->
     <visual name="R_EE_grip_disc_visual">
       <origin
-        xyz="0.008658 0.029717 -0.009909"
-        rpy="1.817146 -0.000000 2.611848" />
+        xyz="0 0.0325 0"
+        rpy="-1.57079632679 0 0" />
       <geometry>
         <cylinder radius="0.03" length="0.01" />
@@ -820,6 +786,6 @@
     <collision name="R_EE_grip_disc_collision">
       <origin
-        xyz="0.008658 0.029717 -0.009909"
-        rpy="1.817146 -0.000000 2.611848" />
+        xyz="0 0.0325 0"
+        rpy="-1.57079632679 0 0" />
       <geometry>
         <cylinder radius="0.03" length="0.01" />
@@ -846,8 +812,8 @@
       velocity="8.5" />
   </joint>
-  <!-- Contact frame at the center and orientation of the existing jmp grip disc. -->
+  <!-- Contact frame at the center and orientation of the neutral grip disc. -->
   <link name="R_grip_frame" />
   <joint name="R_grip_frame_joint" type="fixed">
-    <origin xyz="0.008658 0.029717 -0.009909" rpy="1.817146 0 2.611848" />
+    <origin xyz="0 0.0325 0" rpy="-1.57079632679 0 0" />
     <parent link="R_EE" />
     <child link="R_grip_frame" />
