Commit message: feat: add collision-free wrist pitch joints

File: urdf/dual_arm.urdf (robot description, URDF)
Before this commit: robot dual_arm, 33 links, 32 joints
Links:
- added link L_wrist_pitch, mass 0.15; visual cylinder length=0.03 radius=0.015
- added link R_wrist_pitch, mass 0.15; visual cylinder length=0.03 radius=0.015
Joints:
- added joint L_wrist_pitch_joint: type revolute, parent L_wrist_yaw, child L_wrist_pitch, origin xyz=0 0 -0.12 rpy=0 0 0, axis 0 1 0, limit lower=-0.6 upper=0.6 effort=12 velocity=3
- added joint R_wrist_pitch_joint: type revolute, parent R_wrist_yaw, child R_wrist_pitch, origin xyz=0 0 -0.12 rpy=0 0 0, axis 0 1 0, limit lower=-0.6 upper=0.6 effort=12 velocity=3
- joint L_EE_joint: origin xyz=0 0 -0.15 rpy=0 0 0 -> xyz=0 0 -0.03 rpy=0 0 0; parent L_wrist_yaw -> L_wrist_pitch
- joint L_wrist_ik_joint: parent L_wrist_yaw -> L_wrist_pitch
- joint R_EE_joint: origin xyz=0 0 -0.15 rpy=0 0 0 -> xyz=0 0 -0.03 rpy=0 0 0; parent R_wrist_yaw -> R_wrist_pitch
- joint R_wrist_ik_joint: parent R_wrist_yaw -> R_wrist_pitch

File: urdf/dual_arm.xacro (robot description, xacro)
@@ -364,4 +364,26 @@
     <limit lower="-0.9" upper="0.9" effort="12" velocity="4" />
   </joint>
+  <!-- Pitch axis near the palm.  No collision geometry is used on this small
+       link, avoiding self-contact impulses in the serial wrist chain. -->
+  <link name="L_wrist_pitch">
+    <inertial>
+      <origin xyz="0 0 -0.015" rpy="0 0 0" />
+      <mass value="0.15" />
+      <inertia ixx="0.00015" ixy="0" ixz="0" iyy="0.00015" iyz="0" izz="0.00008" />
+    </inertial>
+    <visual>
+      <origin xyz="0 0 -0.015" rpy="0 0 0" />
+      <geometry><cylinder length="0.03" radius="0.015" /></geometry>
+      <material name="wrist_dark" />
+    </visual>
+  </link>
+  <joint name="L_wrist_pitch_joint" type="revolute">
+    <origin xyz="0 0 -0.12" rpy="0 0 0" />
+    <parent link="L_wrist_yaw" />
+    <child link="L_wrist_pitch" />
+    <axis xyz="0 1 0" />
+    <dynamics damping="1.5" />
+    <limit lower="-0.6" upper="0.6" effort="12" velocity="3" />
+  </joint>
   <link name="L_wrist_ik_frame">
     <inertial>
@@ -373,5 +395,5 @@
   <joint name="L_wrist_ik_joint" type="fixed">
     <origin xyz="0 0 -0.10" rpy="0 0 0" />
-    <parent link="L_wrist_yaw" />
+    <parent link="L_wrist_pitch" />
     <child link="L_wrist_ik_frame" />
   </joint>
@@ -442,8 +464,8 @@
     type="fixed">
     <origin
-      xyz="0 0 -0.15"
+      xyz="0 0 -0.03"
       rpy="0 0 0" />
     <parent
-      link="L_wrist_yaw" />
+      link="L_wrist_pitch" />
     <child
       link="L_EE" />
@@ -721,4 +743,24 @@
     <limit lower="-0.9" upper="0.9" effort="12" velocity="4" />
   </joint>
+  <link name="R_wrist_pitch">
+    <inertial>
+      <origin xyz="0 0 -0.015" rpy="0 0 0" />
+      <mass value="0.15" />
+      <inertia ixx="0.00015" ixy="0" ixz="0" iyy="0.00015" iyz="0" izz="0.00008" />
+    </inertial>
+    <visual>
+      <origin xyz="0 0 -0.015" rpy="0 0 0" />
+      <geometry><cylinder length="0.03" radius="0.015" /></geometry>
+      <material name="wrist_dark" />
+    </visual>
+  </link>
+  <joint name="R_wrist_pitch_joint" type="revolute">
+    <origin xyz="0 0 -0.12" rpy="0 0 0" />
+    <parent link="R_wrist_yaw" />
+    <child link="R_wrist_pitch" />
+    <axis xyz="0 1 0" />
+    <dynamics damping="1.5" />
+    <limit lower="-0.6" upper="0.6" effort="12" velocity="3" />
+  </joint>
   <link name="R_wrist_ik_frame">
     <inertial>
@@ -730,5 +772,5 @@
   <joint name="R_wrist_ik_joint" type="fixed">
     <origin xyz="0 0 -0.10" rpy="0 0 0" />
-    <parent link="R_wrist_yaw" />
+    <parent link="R_wrist_pitch" />
     <child link="R_wrist_ik_frame" />
   </joint>
@@ -797,8 +839,8 @@
     type="fixed">
     <origin
-      xyz="0 0 -0.15"
+      xyz="0 0 -0.03"
       rpy="0 0 0" />
     <parent
-      link="R_wrist_yaw" />
+      link="R_wrist_pitch" />
     <child
       link="R_EE" />
@@ -998,4 +1040,10 @@
     <implicitSpringDamper>true</implicitSpringDamper>
   </gazebo>
+  <gazebo reference="L_wrist_pitch_joint">
+    <implicitSpringDamper>true</implicitSpringDamper>
+  </gazebo>
+  <gazebo reference="R_wrist_pitch_joint">
+    <implicitSpringDamper>true</implicitSpringDamper>
+  </gazebo>
   <!-- 왼쪽/오른쪽 패드 접촉 특성 변경: 기본 kp=1e12(사실상 강체)를 낮춰 접촉 시 임펄스성 반발력을
        줄이고, minDepth로 약간의 침투를 허용해 접촉 안정성을 높인다. L_EE/R_EE 링크(그립 원판이

Commit message: feat: constrain 15DoF IK to arm joints

File: urdf/dual_arm.urdf (robot description, URDF)
Before this commit: robot dual_arm, 35 links, 34 joints
Joints:
- joint L_wrist_ik_joint: origin xyz=0 0 -0.10 rpy=0 0 0 -> xyz=0 0 -0.03 rpy=0 0 0
- joint R_wrist_ik_joint: origin xyz=0 0 -0.10 rpy=0 0 0 -> xyz=0 0 -0.03 rpy=0 0 0

File: urdf/dual_arm.xacro (robot description, xacro)
@@ -394,5 +394,5 @@
   </link>
   <joint name="L_wrist_ik_joint" type="fixed">
-    <origin xyz="0 0 -0.10" rpy="0 0 0" />
+    <origin xyz="0 0 -0.03" rpy="0 0 0" />
     <parent link="L_wrist_pitch" />
     <child link="L_wrist_ik_frame" />
@@ -771,5 +771,5 @@
   </link>
   <joint name="R_wrist_ik_joint" type="fixed">
-    <origin xyz="0 0 -0.10" rpy="0 0 0" />
+    <origin xyz="0 0 -0.03" rpy="0 0 0" />
     <parent link="R_wrist_pitch" />
     <child link="R_wrist_ik_frame" />

Commit message: feat: 손목에 pitch 축 추가, 패드를 pose-independent 원판 마운트로 재구현
배경/문제:
직전 커밋들(054f999, 1712de9)의 yaw 1축 + 사각패드 설계는 Gazebo 실측에서
좌우 접촉 비대칭(L~18.8N, R~0N)으로 그립이 실패했다. 원인은 손바닥 법선이
목표축(월드 Y)에서 X 0.27 + Z 0.45만큼 어긋나는데, 회전축 1개로는 이 다축
오차를 구조적으로 못 없앤다. 같은 admittance-control 계열에서 독립적으로
같은 문제를 풀던 팀원 브랜치(origin/box-lifting)를 확인한 결과, 동일한
결론(yaw만으론 부족)에 도달해 pitch를 추가했고 실제 lift 시도까지 진행한
상태임을 확인함.

검토한 대안과 선택 이유:
- 패드 형상: box-lifting의 원형 패드를 채택(기존 사각 패드 대신). 원판은
  이 저장소의 원래 접촉 물성 튜닝(mu/kp/kd)이 오래 검증된 형상이고, 사각
  패드는 직전 커밋(1712de9)에서 원점을 잘못 잡았을 때 ODE 폭발을 일으킨
  전례가 있어 더 단순하고 안정적인 원판을 우선했다.
- 마운팅 방식: 특정 자세를 오프라인으로 역산한 상수 rpy 대신, box-lifting의
  "EE 로컬 -Y축을 그대로 향하는" pose-independent 마운트(rpy=90,0,0)를
  그대로 채택 - 자세가 바뀔 때마다 재계산해야 했던 근본 문제를 없앤다.
- IK 프레임: pose-independent 마운트 덕에 wrist_ik_frame이 L_EE_joint와
  거의 같은 지점이 되어, 별도 프레임+오프셋 리매핑(직전 계획 Task 1/4)이
  불필요해졌다 - wrist_ik_frame/wrist_ik_joint를 제거하고 L_EE_joint를
  IK가 직접 타겟하도록 되돌린다(Task 3에서 처리).

구현 내용:
L_wrist_pitch_joint/R_wrist_pitch_joint(revolute, y축, ±0.6rad) 추가.
L_EE/R_EE의 콜리전을 사각 박스에서 원판(반경 0.03, 길이 0.01)으로 교체,
마운트를 xyz=(0,∓0.0325,0)/rpy=(±90°,0,0)로 변경(box-lifting과 동일값,
재유도 안 함). L_grip_frame/R_grip_frame을 원판 중심에 고정 프레임으로
추가(Task 4의 동적 스퀴즈축 계산에 사용 예정). L_wrist_ik_frame/
L_wrist_ik_joint 삭제. 4개 손목 관절(yaw+pitch, 양팔) 전부에
implicitSpringDamper 추가 - Task 5 ODE 폭발의 기여 요인으로 추정되는
빠진 설정을 백포트.

결과/검증:
xacro 재생성 후 pinocchio 로드, nq/nv=15 확인, 실제 관절 순서 출력해
기록(다음 태스크에서 이 순서를 그대로 사용). L_EE_joint/R_EE_joint/
L_grip_frame_joint/R_grip_frame_joint 전부 유효한 프레임임을 확인.
Waist_joint 자체는 이번 커밋에서 아예 안 건드림(URDF 리밋 ±0.87rad
그대로) - IK 쪽에서 안 건드리는 건 Task 3에서 검증.

File: urdf/dual_arm.urdf (robot description, URDF)
Before this commit: robot dual_arm, 33 links, 32 joints
Links:
- removed link L_wrist_ik_frame
- removed link R_wrist_ik_frame
- added link L_wrist_pitch, mass 0.15; visual cylinder length=0.03 radius=0.015
- added link R_wrist_pitch, mass 0.15; visual cylinder length=0.03 radius=0.015
- link L_EE: geometry collision cylinder length=0.01 radius=0.03; collision mesh filename=package://dual_arm/meshes/L_EE.STL
- link R_EE: geometry collision cylinder length=0.01 radius=0.03; collision mesh filename=package://dual_arm/meshes/R_EE.STL
Joints:
- removed joint L_grip_joint
- removed joint L_wrist_ik_joint
- removed joint R_grip_joint
- removed joint R_wrist_ik_joint
- added joint L_grip_frame_joint: type fixed, parent L_EE, child L_grip_frame, origin xyz=0 -0.0325 0 rpy=1.57079632679 0 0
- added joint L_wrist_pitch_joint: type revolute, parent L_wrist_yaw, child L_wrist_pitch, origin xyz=0 0 -0.12 rpy=0 0 0, axis 0 1 0, limit lower=-0.6 upper=0.6 effort=12 velocity=3
- added joint R_grip_frame_joint: type fixed, parent R_EE, child R_grip_frame, origin xyz=0 0.0325 0 rpy=-1.57079632679 0 0
- added joint R_wrist_pitch_joint: type revolute, parent R_wrist_yaw, child R_wrist_pitch, origin xyz=0 0 -0.12 rpy=0 0 0, axis 0 1 0, limit lower=-0.6 upper=0.6 effort=12 velocity=3
- joint L_EE_joint: axis (none) -> 0 0 0; limit (none) -> lower=-1.57 upper=1.57 effort=30 velocity=8.5; origin xyz=0 0 -0.15 rpy=0 0 0 -> xyz=0 0 -0.03 rpy=0 0 0; parent L_wrist_yaw -> L_wrist_pitch
- joint L_wrist_yaw_joint: limit lower=-0.9 upper=0.9 effort=12 velocity=4.0 -> lower=-0.9 upper=0.9 effort=12 velocity=4
- joint R_EE_joint: axis (none) -> 0 0 0; limit (none) -> lower=-1.57 upper=1.57 effort=30 velocity=8.5; origin xyz=0 0 -0.15 rpy=0 0 0 -> xyz=0 0 -0.03 rpy=0 0 0; parent R_wrist_yaw -> R_wrist_pitch
- joint R_wrist_yaw_joint: limit lower=-0.9 upper=0.9 effort=12 velocity=4.0 -> lower=-0.9 upper=0.9 effort=12 velocity=4

File: urdf/dual_arm.xacro (robot description, xacro)
@@ -363,19 +363,27 @@
     <axis xyz="0 0 1" />
     <dynamics damping="1" />
-    <limit lower="-0.9" upper="0.9" effort="12" velocity="4.0" />
-  </joint>
-  <!-- Fixed IK-only frame: give it a tiny nonzero inertial or ODE's fixed-joint
-       lumping can become ill-conditioned with a controlled joint upstream. -->
-  <link name="L_wrist_ik_frame">
-    <inertial>
-      <origin xyz="0 0 0" rpy="0 0 0" />
-      <mass value="0.001" />
-      <inertia ixx="1.0E-06" ixy="0" ixz="0" iyy="1.0E-06" iyz="0" izz="1.0E-06" />
-    </inertial>
-  </link>
-  <joint name="L_wrist_ik_joint" type="fixed">
-    <origin xyz="0 0 -0.10" rpy="0 0 0" />
+    <limit lower="-0.9" upper="0.9" effort="12" velocity="4" />
+  </joint>
+  <!-- New: pitch axis near the palm. No collision geometry, same rationale as
+       wrist_yaw (avoid self-contact impulses in the serial wrist chain). -->
+  <link name="L_wrist_pitch">
+    <inertial>
+      <origin xyz="0 0 -0.015" rpy="0 0 0" />
+      <mass value="0.15" />
+      <inertia ixx="0.00015" ixy="0" ixz="0" iyy="0.00015" iyz="0" izz="0.00008" />
+    </inertial>
+    <visual>
+      <origin xyz="0 0 -0.015" rpy="0 0 0" />
+      <geometry><cylinder length="0.03" radius="0.015" /></geometry>
+      <material name="wrist_dark" />
+    </visual>
+  </link>
+  <joint name="L_wrist_pitch_joint" type="revolute">
+    <origin xyz="0 0 -0.12" rpy="0 0 0" />
     <parent link="L_wrist_yaw" />
-    <child link="L_wrist_ik_frame" />
+    <child link="L_wrist_pitch" />
+    <axis xyz="0 1 0" />
+    <dynamics damping="1.5" />
+    <limit lower="-0.6" upper="0.6" effort="12" velocity="3" />
   </joint>
   <link name="L_EE">
@@ -390,27 +398,34 @@
       <material name=""><color rgba="0.298039215686275 0.298039215686275 0.298039215686275 1" /></material>
     </visual>
-    <!-- Single flat palm collision replaces the old STL-mesh + disc-pad combo.
-         Offset/size copied from jys (0.090 x 0.025 x 0.090 box, 3.75cm out in -Y,
-         0.5cm down) - this is a placeholder mount pose to be re-tuned in Task 6
-         against this branch's actual arm geometry, same way the old disc pad
-         needed 3 rounds of offline recomputation. -->
-    <collision name="L_EE_palm_collision">
-      <origin xyz="0 0.0125 -0.005" rpy="0 0 0" />
-      <geometry><box size="0.090 0.025 0.090" /></geometry>
-    </collision>
-    <visual name="L_EE_grip_pad_visual">
-      <origin xyz="0 0.0125 -0.005" rpy="0 0 0" />
-      <geometry><box size="0.090 0.025 0.090" /></geometry>
-      <material name="grip_pad_visual_dark"><color rgba="0.12 0.12 0.12 1" /></material>
-    </visual>
+    <collision>
+      <origin xyz="0 0 0" rpy="0 0 0" />
+      <geometry><mesh filename="package://dual_arm/meshes/L_EE.STL" /></geometry>
+    </collision>
+    <!-- Pose-independent grip pad: normal is exactly the EE local -Y axis. No
+         world-frame IK pose is baked into this geometry; wrist compliance
+         (2 DOF, not 1) does the real-time aligning. Values copied verbatim
+         from origin/box-lifting, do not re-derive. -->
+    <visual name="L_EE_grip_disc_visual">
+      <origin xyz="0 -0.0325 0" rpy="1.57079632679 0 0" />
+      <geometry><cylinder radius="0.03" length="0.01" /></geometry>
+      <material name="grip_pad_orange"><color rgba="1.0 0.5 0.0 1" /></material>
+    </visual>
+    <collision name="L_EE_grip_disc_collision">
+      <origin xyz="0 -0.0325 0" rpy="1.57079632679 0 0" />
+      <geometry><cylinder radius="0.03" length="0.01" /></geometry>
+    </collision>
   </link>
   <joint name="L_EE_joint" type="fixed">
-    <origin xyz="0 0 -0.15" rpy="0 0 0" />
-    <parent link="L_wrist_yaw" />
+    <origin xyz="0 0 -0.03" rpy="0 0 0" />
+    <parent link="L_wrist_pitch" />
     <child link="L_EE" />
-  </joint>
+    <axis xyz="0 0 0" />
+    <dynamics damping="1" />
+    <limit lower="-1.57" upper="1.57" effort="30" velocity="8.5" />
+  </joint>
+  <!-- Contact frame at the center/orientation of the neutral grip disc -->
   <link name="L_grip_frame" />
-  <joint name="L_grip_joint" type="fixed">
-    <origin xyz="0 -0.0375 -0.005" rpy="0 0 0" />
+  <joint name="L_grip_frame_joint" type="fixed">
+    <origin xyz="0 -0.0325 0" rpy="1.57079632679 0 0" />
     <parent link="L_EE" />
     <child link="L_grip_frame" />
@@ -673,19 +688,25 @@
     <axis xyz="0 0 1" />
     <dynamics damping="1" />
-    <limit lower="-0.9" upper="0.9" effort="12" velocity="4.0" />
-  </joint>
-  <!-- Fixed IK-only frame: give it a tiny nonzero inertial or ODE's fixed-joint
-       lumping can become ill-conditioned with a controlled joint upstream. -->
-  <link name="R_wrist_ik_frame">
-    <inertial>
-      <origin xyz="0 0 0" rpy="0 0 0" />
-      <mass value="0.001" />
-      <inertia ixx="1.0E-06" ixy="0" ixz="0" iyy="1.0E-06" iyz="0" izz="1.0E-06" />
-    </inertial>
-  </link>
-  <joint name="R_wrist_ik_joint" type="fixed">
-    <origin xyz="0 0 -0.10" rpy="0 0 0" />
+    <limit lower="-0.9" upper="0.9" effort="12" velocity="4" />
+  </joint>
+  <link name="R_wrist_pitch">
+    <inertial>
+      <origin xyz="0 0 -0.015" rpy="0 0 0" />
+      <mass value="0.15" />
+      <inertia ixx="0.00015" ixy="0" ixz="0" iyy="0.00015" iyz="0" izz="0.00008" />
+    </inertial>
+    <visual>
+      <origin xyz="0 0 -0.015" rpy="0 0 0" />
+      <geometry><cylinder length="0.03" radius="0.015" /></geometry>
+      <material name="wrist_dark" />
+    </visual>
+  </link>
+  <joint name="R_wrist_pitch_joint" type="revolute">
+    <origin xyz="0 0 -0.12" rpy="0 0 0" />
     <parent link="R_wrist_yaw" />
-    <child link="R_wrist_ik_frame" />
+    <child link="R_wrist_pitch" />
+    <axis xyz="0 1 0" />
+    <dynamics damping="1.5" />
+    <limit lower="-0.6" upper="0.6" effort="12" velocity="3" />
   </joint>
   <link name="R_EE">
@@ -700,27 +721,29 @@
       <material name=""><color rgba="0.298039215686275 0.298039215686275 0.298039215686275 1" /></material>
     </visual>
-    <!-- Single flat palm collision replaces the old STL-mesh + disc-pad combo.
-         Offset/size copied from jys (0.090 x 0.025 x 0.090 box, 3.75cm out in +Y,
-         0.5cm down) - this is a placeholder mount pose to be re-tuned in Task 6
-         against this branch's actual arm geometry, same way the old disc pad
-         needed 3 rounds of offline recomputation. -->
-    <collision name="R_EE_palm_collision">
-      <origin xyz="0 -0.0125 -0.005" rpy="0 0 0" />
-      <geometry><box size="0.090 0.025 0.090" /></geometry>
-    </collision>
-    <visual name="R_EE_grip_pad_visual">
-      <origin xyz="0 -0.0125 -0.005" rpy="0 0 0" />
-      <geometry><box size="0.090 0.025 0.090" /></geometry>
-      <material name="grip_pad_visual_dark"><color rgba="0.12 0.12 0.12 1" /></material>
-    </visual>
+    <collision>
+      <origin xyz="0 0 0" rpy="0 0 0" />
+      <geometry><mesh filename="package://dual_arm/meshes/R_EE.STL" /></geometry>
+    </collision>
+    <visual name="R_EE_grip_disc_visual">
+      <origin xyz="0 0.0325 0" rpy="-1.57079632679 0 0" />
+      <geometry><cylinder radius="0.03" length="0.01" /></geometry>
+      <material name="grip_pad_orange"><color rgba="1.0 0.5 0.0 1" /></material>
+    </visual>
+    <collision name="R_EE_grip_disc_collision">
+      <origin xyz="0 0.0325 0" rpy="-1.57079632679 0 0" />
+      <geometry><cylinder radius="0.03" length="0.01" /></geometry>
+    </collision>
   </link>
   <joint name="R_EE_joint" type="fixed">
-    <origin xyz="0 0 -0.15" rpy="0 0 0" />
-    <parent link="R_wrist_yaw" />
+    <origin xyz="0 0 -0.03" rpy="0 0 0" />
+    <parent link="R_wrist_pitch" />
     <child link="R_EE" />
+    <axis xyz="0 0 0" />
+    <dynamics damping="1" />
+    <limit lower="-1.57" upper="1.57" effort="30" velocity="8.5" />
   </joint>
   <link name="R_grip_frame" />
-  <joint name="R_grip_joint" type="fixed">
-    <origin xyz="0 0.0375 -0.005" rpy="0 0 0" />
+  <joint name="R_grip_frame_joint" type="fixed">
+    <origin xyz="0 0.0325 0" rpy="-1.57079632679 0 0" />
     <parent link="R_EE" />
     <child link="R_grip_frame" />
@@ -918,4 +941,11 @@
     <maxVel>0.0</maxVel>
   </gazebo>
+  <!-- Use ODE's implicit damping for the wrist axes; explicit-only damping
+       under contact-driven torque spikes contributed to the ODE explosion
+       seen in the previous plan's Task 5 Gazebo test. -->
+  <gazebo reference="L_wrist_yaw_joint"><implicitSpringDamper>true</implicitSpringDamper></gazebo>
+  <gazebo reference="R_wrist_yaw_joint"><implicitSpringDamper>true</implicitSpringDamper></gazebo>
+  <gazebo reference="L_wrist_pitch_joint"><implicitSpringDamper>true</implicitSpringDamper></gazebo>
+  <gazebo reference="R_wrist_pitch_joint"><implicitSpringDamper>true</implicitSpringDamper></gazebo>
   <!-- gazebo_ros_ft_sensor: L_EE_joint/R_EE_joint에 걸리는 반력을 각각
        /dual_arm/left_ft_sensor, /dual_arm/right_ft_sensor (geometry_msgs/WrenchStamped)로 발행. -->

Commit message: fix: orient wrist flexion axis across palm normal
배경/문제:
수동 손목 정렬 시험에서 물체를 들 수는 있었지만 손바닥 전체가 면에 닿지 않고 물체가 크게 기울었다. URDF를 확인한 결과 wrist_pitch_joint의 Y축이 손바닥 접촉면 법선인 local Y와 평행해, 해당 관절이 접촉면을 기울이지 못하고 원형 패드를 면 안에서 회전시키는 역할만 하고 있었다.

검토한 대안과 선택 이유:
현재 Z축 yaw와 Y축 pitch를 유지한 채 제어만 조정하는 방법은 두 번째 관절이 패드 법선 정렬에 기구학적으로 기여하지 못하므로 제외했다. 손바닥 법선 Y에 서로 수직인 Z축과 X축 조합이 접촉면의 두 방향 기울기를 만들 수 있어 두 번째 축을 X로 변경했다.

구현 내용:
좌우 L/R_wrist_pitch_joint의 axis를 0 1 0에서 1 0 0으로 변경했다. xacro 원본과 저장소에 포함된 생성 URDF를 함께 갱신하고, 왼손 축의 설명을 손바닥 법선과의 관계가 드러나도록 수정했다. 관절 이름과 limit, damping, transmission 및 제어 인덱스는 유지했다.

결과/검증:
xacro --inorder로 생성한 URDF에서 좌우 wrist_pitch_joint 축이 모두 1 0 0임을 확인했다. git diff --check를 통과했고 catkin_make --pkg dual_arm -j2에서 dual_arm_main과 dual_arm_command 빌드가 성공했다. 변경된 접촉면 정렬과 파지력의 Gazebo 런타임 검증은 다음 실행에서 수행해야 한다.

File: urdf/dual_arm.urdf (robot description, URDF)
Before this commit: robot dual_arm, 35 links, 34 joints
Joints:
- joint L_elbow_joint: axis 0 1 0 -> 1 0 0
- joint L_shoulder_pitch_joint: axis 0 1 0 -> 1 0 0

File: urdf/dual_arm.xacro (robot description, xacro)
@@ -364,6 +364,7 @@
     <limit lower="-0.9" upper="0.9" effort="12" velocity="4" />
   </joint>
-  <!-- Pitch axis near the palm.  No collision geometry is used on this small
-       link, avoiding self-contact impulses in the serial wrist chain. -->
+  <!-- Flexion axis near the palm. The palm normal is local Y, so this second
+       wrist axis is local X to tilt the contact face. No collision geometry
+       is used on this small link, avoiding serial-chain self contact. -->
   <link name="L_wrist_pitch">
     <inertial>
@@ -382,5 +383,5 @@
     <parent link="L_wrist_yaw" />
     <child link="L_wrist_pitch" />
-    <axis xyz="0 1 0" />
+    <axis xyz="1 0 0" />
     <dynamics damping="1.5" />
     <limit lower="-0.6" upper="0.6" effort="12" velocity="3" />
@@ -759,5 +760,5 @@
     <parent link="R_wrist_yaw" />
     <child link="R_wrist_pitch" />
-    <axis xyz="0 1 0" />
+    <axis xyz="1 0 0" />
     <dynamics damping="1.5" />
     <limit lower="-0.6" upper="0.6" effort="12" velocity="3" />
