Commit message: feat: 손바닥 전후 굽힘 손목 자유도 재설계
13DoF 중립 손바닥 상태에서 좌우 wrist_pitch link와 관절을 yaw와 EE 사이에 추가했다. 손바닥 접촉면 법선인 local Y와 수직인 local X를 회전축으로 사용해 패드를 면 안에서 회전시키지 않고 앞뒤로 젖힐 수 있게 했다.

elbow-to-EE 길이 0.30m와 기존 손바닥/F/T 구조를 유지했으며 작은 flexion link는 collision 없이 구성했다. xacro, check_urdf 및 catkin 빌드를 통과했다.

spawn-only 15초 시험에서 상태는 모두 finite였고 flexion 최대 드리프트 0.000613rad, 최대 속도 0.000930rad/s였다. 물리를 정지한 상태에서 좌우 관절에 +0.45rad와 -0.45rad를 적용해 손바닥 전후 굽힘 방향도 GUI로 확인했다.

File: urdf/dual_arm.urdf (robot description, URDF)
Before this commit: robot dual_arm, 33 links, 32 joints
Links:
- added link L_wrist_pitch, mass 0.15; visual cylinder length=0.03 radius=0.015
- added link R_wrist_pitch, mass 0.15; visual cylinder length=0.03 radius=0.015
Joints:
- added joint L_wrist_pitch_joint: type revolute, parent L_wrist_yaw, child L_wrist_pitch, origin xyz=0 0 -0.12 rpy=0 0 0, axis 1 0 0, limit lower=-0.6 upper=0.6 effort=12 velocity=3
- added joint R_wrist_pitch_joint: type revolute, parent R_wrist_yaw, child R_wrist_pitch, origin xyz=0 0 -0.12 rpy=0 0 0, axis 0 1 0, limit lower=-0.6 upper=0.6 effort=12 velocity=3
- joint L_EE_joint: origin xyz=0 0 -0.15 rpy=0 0 0 -> xyz=0 0 -0.03 rpy=0 0 0; parent L_wrist_yaw -> L_wrist_pitch
- joint L_wrist_ik_joint: parent L_wrist_yaw -> L_wrist_pitch
- joint R_EE_joint: origin xyz=0 0 -0.15 rpy=0 0 0 -> xyz=0 0 -0.03 rpy=0 0 0; parent R_wrist_yaw -> R_wrist_pitch
- joint R_shoulder_pitch_joint: axis 0 1 0 -> 1 0 0
- joint R_wrist_ik_joint: parent R_wrist_yaw -> R_wrist_pitch

File: urdf/dual_arm.xacro (robot description, xacro)
@@ -364,4 +364,26 @@
     <limit lower="-0.9" upper="0.9" effort="12" velocity="4" />
   </joint>
+  <!-- Palm flexion axis near the palm. The contact normal is local Y, so the
+       local X axis tilts the palm forward/back instead of spinning it in-plane. -->
+  <link name="L_wrist_pitch">
+    <inertial>
+      <origin xyz="0 0 -0.015" rpy="0 0 0" />
+      <mass value="0.15" />
+      <inertia ixx="0.00015" ixy="0" ixz="0" iyy="0.00015" iyz="0" izz="0.00008" />
+    </inertial>
+    <visual>
+      <origin xyz="0 0 -0.015" rpy="0 0 0" />
+      <geometry><cylinder length="0.03" radius="0.015" /></geometry>
+      <material name="wrist_dark" />
+    </visual>
+  </link>
+  <joint name="L_wrist_pitch_joint" type="revolute">
+    <origin xyz="0 0 -0.12" rpy="0 0 0" />
+    <parent link="L_wrist_yaw" />
+    <child link="L_wrist_pitch" />
+    <axis xyz="1 0 0" />
+    <dynamics damping="1.5" />
+    <limit lower="-0.6" upper="0.6" effort="12" velocity="3" />
+  </joint>
   <link name="L_wrist_ik_frame">
     <inertial>
@@ -373,5 +395,5 @@
   <joint name="L_wrist_ik_joint" type="fixed">
     <origin xyz="0 0 -0.10" rpy="0 0 0" />
-    <parent link="L_wrist_yaw" />
+    <parent link="L_wrist_pitch" />
     <child link="L_wrist_ik_frame" />
   </joint>
@@ -442,8 +464,8 @@
     type="fixed">
     <origin
-      xyz="0 0 -0.15"
+      xyz="0 0 -0.03"
       rpy="0 0 0" />
     <parent
-      link="L_wrist_yaw" />
+      link="L_wrist_pitch" />
     <child
       link="L_EE" />
@@ -721,4 +743,24 @@
     <limit lower="-0.9" upper="0.9" effort="12" velocity="4" />
   </joint>
+  <link name="R_wrist_pitch">
+    <inertial>
+      <origin xyz="0 0 -0.015" rpy="0 0 0" />
+      <mass value="0.15" />
+      <inertia ixx="0.00015" ixy="0" ixz="0" iyy="0.00015" iyz="0" izz="0.00008" />
+    </inertial>
+    <visual>
+      <origin xyz="0 0 -0.015" rpy="0 0 0" />
+      <geometry><cylinder length="0.03" radius="0.015" /></geometry>
+      <material name="wrist_dark" />
+    </visual>
+  </link>
+  <joint name="R_wrist_pitch_joint" type="revolute">
+    <origin xyz="0 0 -0.12" rpy="0 0 0" />
+    <parent link="R_wrist_yaw" />
+    <child link="R_wrist_pitch" />
+    <axis xyz="1 0 0" />
+    <dynamics damping="1.5" />
+    <limit lower="-0.6" upper="0.6" effort="12" velocity="3" />
+  </joint>
   <link name="R_wrist_ik_frame">
     <inertial>
@@ -730,5 +772,5 @@
   <joint name="R_wrist_ik_joint" type="fixed">
     <origin xyz="0 0 -0.10" rpy="0 0 0" />
-    <parent link="R_wrist_yaw" />
+    <parent link="R_wrist_pitch" />
     <child link="R_wrist_ik_frame" />
   </joint>
@@ -797,8 +839,8 @@
     type="fixed">
     <origin
-      xyz="0 0 -0.15"
+      xyz="0 0 -0.03"
       rpy="0 0 0" />
     <parent
-      link="R_wrist_yaw" />
+      link="R_wrist_pitch" />
     <child
       link="R_EE" />
@@ -998,4 +1040,10 @@
     <implicitSpringDamper>true</implicitSpringDamper>
   </gazebo>
+  <gazebo reference="L_wrist_pitch_joint">
+    <implicitSpringDamper>true</implicitSpringDamper>
+  </gazebo>
+  <gazebo reference="R_wrist_pitch_joint">
+    <implicitSpringDamper>true</implicitSpringDamper>
+  </gazebo>
   <!-- 왼쪽/오른쪽 패드 접촉 특성 변경: 기본 kp=1e12(사실상 강체)를 낮춰 접촉 시 임펄스성 반발력을
        줄이고, minDepth로 약간의 침투를 허용해 접촉 안정성을 높인다. L_EE/R_EE 링크(그립 원판이

Commit message: fix: 오른팔 pitch 모델 축 불일치 수정
Gazebo가 사용하는 xacro는 오른쪽 shoulder pitch를 Y축으로 정의하지만 Pinocchio 입력 URDF만 X축으로 남아 있었다. URDF 축을 Y축으로 맞춰 중력 보상과 IK가 실제 물리 관절과 동일한 모델을 사용하도록 한다.\n\n검증:\n- GUI 12초 안정화 후 최종 최대 관절 속도 2.59e-5 rad/s\n- 좌우 안전 목표 관절 오차 약 0.4mrad 이하(오른 손목 pitch 제외 14mrad)\n- Mission4 IK 좌 0.233mm, 우 0.210mm, torso error 0

File: urdf/dual_arm.urdf (robot description, URDF)
Before this commit: robot dual_arm, 35 links, 34 joints
Joints:
- joint R_shoulder_pitch_joint: axis 1 0 0 -> 0 1 0
