Commit message: fix: 손목 pitch 조인트 회전축을 로컬 Y에서 X로 변경
배경/문제:
L_wrist_pitch_joint/R_wrist_pitch_joint의 axis가 로컬 Y축(0 1 0)으로 되어 있었는데,
그립패드의 접촉 법선(스퀴즈 방향)도 동일하게 EE 로컬 Y축이다(F/T force.y가 스퀴즈력을
나타낸다는 기존 설계와 main.cpp의 손목 정렬 로직 참고). 즉 pitch 조인트 회전축과 접촉
법선 축이 겹쳐 있어서, 이 조인트가 움직여도 패드가 물체 표면에 대해 기울어지는 게
아니라 접촉면 법선을 축으로 제자리에서 헛도는 상태였다 - "표면에 맞춰 기울어지는
컴플라이언스"라는 원래 의도한 기능을 못 하고 있었을 가능성이 높았다.

검토한 대안과 선택 이유:
GitHub jy02sung/URP_summer_26의 vertical_lift_final 브랜치와 코드를 비교하는 과정에서
이 축이 로컬 X축(1 0 0)으로 되어 있는 것을 발견했고, 그 브랜치 주석에 "접촉 법선이
로컬 Y라서 로컬 X축이어야 패드를 앞뒤로 기울이지, 그 자리에서 헛돌지 않는다"는 설명이
있어 이 branch의 값이 우리 branch의 버그를 고친 것으로 판단했다. 다른 대안(예: pitch
조인트 자체를 재배치)은 검토하지 않았다 - 축 값만 바꾸는 게 가장 국소적이고 명확한 수정.

구현 내용:
urdf/dual_arm.xacro와 urdf/dual_arm.urdf 양쪽에서 L_wrist_pitch_joint, R_wrist_pitch_joint의
<axis>를 "0 1 0"에서 "1 0 0"으로 변경. xacro는 Gazebo/RViz가 런타임에 xacro 커맨드로
robot_description을 생성할 때 쓰고, urdf는 main.cpp가 pinocchio로 직접 로드하는 정적
파일이라(ros::package::getPath + "/urdf/dual_arm.urdf") 두 파일 모두 동일하게 수정해야
IK와 시뮬레이션이 같은 기구학을 보게 된다.

결과/검증:
catkin_make --only-pkg-with-deps dual_arm 빌드 성공 확인. urdf/xacro는 컴파일 대상이
아니라 런타임 리소스라 재컴파일은 필요 없고, 다음 Gazebo 실행부터 반영된다. 이후 실행한
force_log CSV에서 이번 세션의 좌우 스퀴즈력 비대칭 방향이 과거 RETRY_FROM_88PCT.md 기록과
반대로 나타난 것(R이 L보다 안정적)을 관찰했는데, 이 축 수정이 원인일 가능성이 있어 보이나
반복 실행으로 재현성 검증은 아직 못 했다 - 다음 세션에서 확인 필요.

Co-Authored-By: Claude Sonnet 5 <noreply@anthropic.com>

File: urdf/dual_arm.urdf (robot description, URDF)
Before this commit: robot dual_arm, 33 links, 32 joints
Joints:
- joint L_wrist_pitch_joint: axis 0 1 0 -> 1 0 0
- joint R_wrist_pitch_joint: axis 0 1 0 -> 1 0 0

File: urdf/dual_arm.xacro (robot description, xacro)
@@ -383,5 +383,5 @@
     <parent link="L_wrist_yaw" />
     <child link="L_wrist_pitch" />
-    <axis xyz="0 1 0" />
+    <axis xyz="1 0 0" />
     <dynamics damping="1.5" />
     <limit lower="-0.6" upper="0.6" effort="12" velocity="3" />
@@ -706,5 +706,5 @@
     <parent link="R_wrist_yaw" />
     <child link="R_wrist_pitch" />
-    <axis xyz="0 1 0" />
+    <axis xyz="1 0 0" />
     <dynamics damping="1.5" />
     <limit lower="-0.6" upper="0.6" effort="12" velocity="3" />
